File: hw/controller.kicad_sch (KiCad schematic)
At the start: 0 parts

Commit message: working on documentation, design methmethodology, sizing, layout
Parts:
- added C201: 100nF, Capacitor_SMD:C_0402_1005Metric, symbol Device:C_Small
- added D202: BLUE, LED_SMD:LED_0805_2012Metric, symbol Device:LED
- added D203: YELLOW, LED_SMD:LED_0805_2012Metric, symbol Device:LED
- added D204: RED, LED_SMD:LED_0805_2012Metric, symbol Device:LED
- added J201: 1935776, 1935776, symbol 1935776:1935776
- added R201, R202, R203: 330, Resistor_SMD:R_0805_2012Metric, symbol Device:R
- added SW201: SW_Push, Button_Switch_THT:SW_PUSH_6mm, symbol Switch:SW_Push
- added TP201: 3.3V TP, TestPoint:TestPoint_Pad_2.0x2.0mm, symbol Connector:TestPoint
- added TP202: 12V TP, TestPoint:TestPoint_Pad_2.0x2.0mm, symbol Connector:TestPoint
- added TP203: 5V TP, TestPoint:TestPoint_Pad_2.0x2.0mm, symbol Connector:TestPoint
- added TP204: GND MCU TP, TestPoint:TestPoint_Pad_2.0x2.0mm, symbol Connector:TestPoint
- added U201: MCU_Nucleo_L432KC, mppt:MODULE_NUCLEO-L432KC, symbol MPPT:MCU_Nucleo_L432KC
Connections:
- new net: D202.2 (A), R203.1
- new net: D203.2 (A), R202.1
- new net: D204.2 (A), R201.1
- new net +12V: C201.1, J201.1, TP202.1, U201.30 (VIN)
- new net +3.3V: TP201.1, U201.17 (+3V3)
- new net +5V: TP203.1, U201.27 (+5V)
- new net ARR_CURRENT: U201.22 (A3)
- new net ARR_VOLTAGE: U201.23 (A4)
- new net BATT_CURRENT: U201.24 (A5)
- new net BATT_VOLTAGE: U201.25 (A6)
- new net Error: R201.2, U201.15 (D12)
- new net GND: C201.2, D202.1 (K), D203.1 (K), D204.1 (K), J201.2, SW201.1, TP204.1, U201.29 (GND), U201.4 (GND)
- new net Heartbeat: R203.2, U201.13 (D10)
- new net PWM: U201.20 (A1)
- new net Reset: SW201.2, U201.28 (RST), U201.3 (RST)
- new net Tracking: R202.2, U201.14 (D11)
- no-connect marks 0 -> 15

Commit message: parts of gate driver
Connections:
- net PWM_EN: now reaches U201.19 (A0)
- no-connect marks 15 -> 14
Changed lines of the file:
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@@
   (no_connect (at 140.97 72.39))
   (no_connect (at 140.97 74.93))
-  (no_connect (at 166.37 100.33))
   (no_connect (at 140.97 97.79))
   (no_connect (at 166.37 107.95))
@@
     (effects (font (size 1.27 1.27)) (justify left))
   )
+  (hierarchical_label "PWM_EN" (shape input) (at 166.37 100.33 0) (fields_autoplaced)
+    (effects (font (size 1.27 1.27)) (justify left))
+  )

Commit message: layout revision this one is cursed
Changed lines of the file:
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@@
   (junction (at 190.5 72.39) (diameter 0) (color 0 0 0 0)
   )
+  (junction (at 182.88 72.39) (diameter 0) (color 0 0 0 0)
+  )
   (junction (at 175.26 80.01) (diameter 0) (color 0 0 0 0)
+  )
+  (junction (at 184.15 77.47) (diameter 0) (color 0 0 0 0)
   )
   (junction (at 190.5 78.74) (diameter 0) (color 0 0 0 0)
@@
     (stroke (width 0) (type default))
   )
-  (wire (pts (xy 179.07 77.47) (xy 190.5 77.47))
+  (wire (pts (xy 179.07 77.47) (xy 184.15 77.47))
     (stroke (width 0) (type default))
   )
@@
     (stroke (width 0) (type default))
   )
-  (wire (pts (xy 175.26 72.39) (xy 190.5 72.39))
+  (wire (pts (xy 175.26 72.39) (xy 182.88 72.39))
     (stroke (width 0) (type default))
   )
@@
     (stroke (width 0) (type default))
   )
+  (wire (pts (xy 184.15 77.47) (xy 190.5 77.47))
+    (stroke (width 0) (type default))
+  )
   (wire (pts (xy 105.41 83.82) (xy 105.41 85.09))
     (stroke (width 0) (type default))
@@
   )
   (wire (pts (xy 120.65 80.01) (xy 120.65 82.55))
+    (stroke (width 0) (type default))
+  )
+  (wire (pts (xy 182.88 72.39) (xy 190.5 72.39))
     (stroke (width 0) (type default))
   )
@@
     )
   )
+  (symbol (lib_id "power:PWR_FLAG") (at 182.88 72.39 0) (unit 1)
+    (in_bom yes) (on_board yes) (dnp no) (fields_autoplaced)
+    (property "Reference" "#FLG0201" (at 182.88 70.485 0)
+      (effects (font (size 1.27 1.27)) hide)
+    )
+    (property "Value" "PWR_FLAG" (at 182.88 68.58 0)
+      (effects (font (size 1.27 1.27)))
+    )
+    (property "Footprint" "" (at 182.88 72.39 0)
+      (effects (font (size 1.27 1.27)) hide)
+    )
+    (property "Datasheet" "~" (at 182.88 72.39 0)
+      (effects (font (size 1.27 1.27)) hide)
+    )
+    (pin "1")
+    (instances
+      (project "mppt"
+        (path "/06fd3a42-664d-41bc-bf0f-b5ee0ddcc902/90f57858-b3ac-468b-8edb-acb0ab266950"
+          (reference "#FLG0201") (unit 1)
+        )
+      )
+    )
+  )
   (symbol (lib_id "power:GND") (at 82.55 100.33 0) (unit 1)
     (in_bom yes) (on_board yes) (dnp no) (fields_autoplaced)
@@
         )
       )
+    )
+  )
+  (symbol (lib_id "power:PWR_FLAG") (at 184.15 77.47 0) (unit 1)
+    (in_bom yes) (on_board yes) (dnp no) (fields_autoplaced)
+    (property "Reference" "#FLG0202" (at 184.15 75.565 0)
+      (effects (font (size 1.27 1.27)) hide)
+    )
+    (property "Value" "PWR_FLAG" (at 184.15 73.66 0)
+      (effects (font (size 1.27 1.27)))
+    )
+    (property "Footprint" "" (at 184.15 77.47 0)
+      (effects (font (size 1.27 1.27)) hide)
+    )
+    (property "Datasheet" "~" (at 184.15 77.47 0)
+      (effects (font (size 1.27 1.27)) hide)
+    )
+    (pin "1")
+    (instances
+      (project "mppt"
+        (path "/06fd3a42-664d-41bc-bf0f-b5ee0ddcc902/90f57858-b3ac-468b-8edb-acb0ab266950"
+          (reference "#FLG0202") (unit 1)
+        )
+      )

Commit message: slight bom updates
Parts:
- C201: In Stock? (none) -> Y; Mfr PN (none) -> CL21B104KCFNNNE; Projected Cost (none) -> 0.008
- D202: In Stock? (none) -> Y; Mfr PN (none) -> SZYY0805B; Projected Cost (none) -> 0.0129
- D203: In Stock? (none) -> Y; Mfr PN (none) -> SZYY0805YG; Projected Cost (none) -> 0.0123
- D204: In stock? (none) -> Y; Mfr PN (none) -> NCD0805R1; Projected Cost (none) -> 0.0114
- J201: In Stock? (none) -> Y; Projected Cost (none) -> 0.59
- R201, R202, R203: In Stock? (none) -> Y
- U201: In Stock? (none) -> N/A
Changed lines of the file:
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@@
       (effects (font (size 1 1)) hide)
+    )
+    (property "In Stock?" "Y" (at 105.41 88.9 90)
+      (effects (font (size 1.27 1.27)) hide)
     )
     (pin "1")
@@
     (property "Datasheet" "https://www.mouser.com/datasheet/2/389/nucleo-f031k6-1484037.pdf" (at 153.67 97.79 0)
       (effects (font (size 1.524 1.524)) hide)
+    )
+    (property "In Stock?" "N/A" (at 153.67 90.17 0)
+      (effects (font (size 1.27 1.27)) hide)
     )
     (pin "1")
@@
       (effects (font (size 1.27 1.27)) hide)
     )
+    (property "Mfr PN" "SZYY0805YG" (at 93.98 96.52 90)
+      (effects (font (size 1.27 1.27)) hide)
+    )
+    (property "Projected Cost" "0.0123" (at 93.98 96.52 90)
+      (effects (font (size 1.27 1.27)) hide)
+    )
+    (property "In Stock?" "Y" (at 93.98 96.52 90)
+      (effects (font (size 1.27 1.27)) hide)
+    )
     (pin "1")
     (pin "2")
@@
     )
     (property "Datasheet" "~" (at 82.55 96.52 0)
+      (effects (font (size 1.27 1.27)) hide)
+    )
+    (property "Mfr PN" "NCD0805R1" (at 82.55 96.52 90)
+      (effects (font (size 1.27 1.27)) hide)
+    )
+    (property "Projected Cost" "0.0114" (at 82.55 96.52 90)
+      (effects (font (size 1.27 1.27)) hide)
+    )
+    (property "In stock?" "Y" (at 82.55 96.52 90)
       (effects (font (size 1.27 1.27)) hide)
     )
@@
       (effects (font (size 1 1)) hide)
     )
+    (property "In Stock?" "Y" (at 93.98 88.9 90)
+      (effects (font (size 1.27 1.27)) hide)
+    )
     (pin "1")
     (pin "2")
@@
       (effects (font (size 1.27 1.27)) hide)
     )
+    (property "Mfr PN" "CL21B104KCFNNNE" (at 190.5 74.93 0)
+      (effects (font (size 1.27 1.27)) hide)
+    )
+    (property "In Stock?" "Y" (at 190.5 74.93 0)
+      (effects (font (size 1.27 1.27)) hide)
+    )
+    (property "Projected Cost" "0.008" (at 190.5 74.93 0)
+      (effects (font (size 1.27 1.27)) hide)
+    )
     (pin "1")
     (pin "2")
@@
     (property "MOUSER_PRICE-STOCK" "https://www.mouser.co.uk/ProductDetail/Phoenix-Contact/1935776?qs=gjk32EaArKJ3oesOAo3TWA%3D%3D" (at 203.2 72.39 0)
       (effects (font (size 1.27 1.27)) (justify bottom) hide)
+    )
+    (property "Projected Cost" "0.59" (at 203.2 72.39 0)
+      (effects (font (size 1.27 1.27)) hide)
+    )
+    (property "In Stock?" "Y" (at 203.2 72.39 0)
+      (effects (font (size 1.27 1.27)) hide)
     )
     (pin "1")
@@
       (effects (font (size 1 1)) hide)
     )
+    (property "In Stock?" "Y" (at 82.55 88.9 90)
+      (effects (font (size 1.27 1.27)) hide)
+    )
     (pin "1")
     (pin "2")
@@
       (effects (font (size 1.27 1.27)) hide)
     )
+    (property "Mfr PN" "SZYY0805B" (at 105.41 96.52 90)
+      (effects (font (size 1.27 1.27)) hide)
+    )
+    (property "Projected Cost" "0.0129" (at 105.41 96.52 90)
+      (effects (font (size 1.27 1.27)) hide)
+    )
+    (property "In Stock?" "Y" (at 105.41 96.52 90)
+      (effects (font (size 1.27 1.27)) hide)
+    )

Commit message: revision of PCB layout
Connections:
- net ARR_CURRENT: now also U201.23 (A4); no longer U201.22 (A3)
- net ARR_VOLTAGE: now also U201.22 (A3); no longer U201.23 (A4)
- net Error: now also U201.5 (D2); no longer U201.15 (D12)
- net Heartbeat: now also U201.1 (D1); no longer U201.13 (D10)
- net Tracking: now also U201.2 (D0); no longer U201.14 (D11)
Changed lines of the file:
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@@
   (no_connect (at 166.37 95.25))
   (no_connect (at 140.97 92.71))
-  (no_connect (at 140.97 82.55))
+  (no_connect (at 140.97 105.41))
   (no_connect (at 140.97 95.25))
   (no_connect (at 140.97 100.33))
-  (no_connect (at 140.97 72.39))
-  (no_connect (at 140.97 74.93))
+  (no_connect (at 140.97 102.87))
   (no_connect (at 140.97 97.79))
   (no_connect (at 166.37 107.95))
   (no_connect (at 166.37 82.55))
+  (no_connect (at 140.97 107.95))
   (no_connect (at 140.97 85.09))
   (no_connect (at 140.97 87.63))
   (no_connect (at 166.37 102.87))
   (wire (pts (xy 93.98 83.82) (xy 93.98 85.09))
+    (stroke (width 0) (type default))
+  )
+  (wire (pts (xy 130.81 74.93) (xy 140.97 74.93))
     (stroke (width 0) (type default))
   )
@@
     (stroke (width 0) (type default))
   )
-  (wire (pts (xy 130.81 102.87) (xy 140.97 102.87))
-    (stroke (width 0) (type default))
-  )
   (wire (pts (xy 82.55 83.82) (xy 82.55 85.09))
     (stroke (width 0) (type default))
@@
   )
   (wire (pts (xy 175.26 72.39) (xy 182.88 72.39))
+    (stroke (width 0) (type default))
+  )
+  (wire (pts (xy 130.81 82.55) (xy 140.97 82.55))
     (stroke (width 0) (type default))
   )
@@
     (stroke (width 0) (type default))
   )
+  (wire (pts (xy 130.81 72.39) (xy 140.97 72.39))
+    (stroke (width 0) (type default))
+  )
   (wire (pts (xy 182.88 72.39) (xy 190.5 72.39))
     (stroke (width 0) (type default))
   )
-  (wire (pts (xy 130.81 107.95) (xy 140.97 107.95))
-    (stroke (width 0) (type default))
-  )
-  (wire (pts (xy 130.81 105.41) (xy 140.97 105.41))
-    (stroke (width 0) (type default))
+  (label "Heartbeat" (at 130.81 72.39 0) (fields_autoplaced)
+    (effects (font (size 1.27 1.27)) (justify left bottom))
   )
   (label "Heartbeat" (at 105.41 83.82 0) (fields_autoplaced)
-    (effects (font (size 1.27 1.27)) (justify left bottom))
-  )
-  (label "Error" (at 130.81 107.95 0) (fields_autoplaced)
     (effects (font (size 1.27 1.27)) (justify left bottom))
   )
@@
     (effects (font (size 1.27 1.27)) (justify left bottom))
   )
-  (label "Tracking" (at 130.81 105.41 0) (fields_autoplaced)
+  (label "Error" (at 130.81 82.55 0) (fields_autoplaced)
     (effects (font (size 1.27 1.27)) (justify left bottom))
   )
@@
     (effects (font (size 1.27 1.27)) (justify left bottom))
   )
-  (label "Heartbeat" (at 130.81 102.87 0) (fields_autoplaced)
+  (label "Tracking" (at 130.81 74.93 0) (fields_autoplaced)
     (effects (font (size 1.27 1.27)) (justify left bottom))
   )
@@
     (effects (font (size 1.27 1.27)) (justify left))
   )
-  (hierarchical_label "ARR_VOLTAGE" (shape input) (at 166.37 90.17 0) (fields_autoplaced)
-    (effects (font (size 1.27 1.27)) (justify left))
-  )
   (hierarchical_label "BATT_CURRENT" (shape input) (at 166.37 87.63 0) (fields_autoplaced)
     (effects (font (size 1.27 1.27)) (justify left))
@@
     (effects (font (size 1.27 1.27)) (justify left))
   )
-  (hierarchical_label "ARR_CURRENT" (shape input) (at 166.37 92.71 0) (fields_autoplaced)
-    (effects (font (size 1.27 1.27)) (justify left))
-  )
   (hierarchical_label "PWM_EN" (shape input) (at 166.37 100.33 0) (fields_autoplaced)
     (effects (font (size 1.27 1.27)) (justify left))
   )
+  (hierarchical_label "ARR_CURRENT" (shape input) (at 166.37 90.17 0) (fields_autoplaced)
+    (effects (font (size 1.27 1.27)) (justify left))
+  )
+  (hierarchical_label "ARR_VOLTAGE" (shape input) (at 166.37 92.71 0) (fields_autoplaced)
+    (effects (font (size 1.27 1.27)) (justify left))
+  )

Commit message: segregating code into design procedures
Parts:
- renumbered D204 to D201, D203 to D202, D202 to D203, TP203 to TP201, TP201 to TP202, TP202 to TP203
Connections:
- net PWM_EN: now also U201.21 (A2); no longer U201.19 (A0)
Changed lines of the file:
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@@
   (junction (at 175.26 72.39) (diameter 0) (color 0 0 0 0)
   )
+  (junction (at 170.18 80.01) (diameter 0) (color 0 0 0 0)
+  )
   (junction (at 177.8 105.41) (diameter 0) (color 0 0 0 0)
   )
@@
   )
   (no_connect (at 140.97 90.17))
-  (no_connect (at 166.37 95.25))
   (no_connect (at 140.97 92.71))
   (no_connect (at 140.97 105.41))
@@
   (no_connect (at 140.97 85.09))
   (no_connect (at 140.97 87.63))
+  (no_connect (at 166.37 100.33))
   (no_connect (at 166.37 102.87))
   (wire (pts (xy 93.98 83.82) (xy 93.98 85.09))
@@
     (stroke (width 0) (type default))
   )
+  (wire (pts (xy 170.18 80.01) (xy 175.26 80.01))
+    (stroke (width 0) (type default))
+  )
   (wire (pts (xy 179.07 77.47) (xy 184.15 77.47))
     (stroke (width 0) (type default))
@@
     (stroke (width 0) (type default))
   )
-  (wire (pts (xy 166.37 80.01) (xy 175.26 80.01))
+  (wire (pts (xy 166.37 80.01) (xy 170.18 80.01))
     (stroke (width 0) (type default))
   )
@@
     (effects (font (size 1.27 1.27)) (justify left))
   )
+  (hierarchical_label "PWM_EN" (shape input) (at 166.37 95.25 0) (fields_autoplaced)
+    (effects (font (size 1.27 1.27)) (justify left))
+  )
   (hierarchical_label "BATT_CURRENT" (shape input) (at 166.37 87.63 0) (fields_autoplaced)
     (effects (font (size 1.27 1.27)) (justify left))
@@
     (effects (font (size 1.27 1.27)) (justify left))
   )
-  (hierarchical_label "PWM_EN" (shape input) (at 166.37 100.33 0) (fields_autoplaced)
-    (effects (font (size 1.27 1.27)) (justify left))
-  )
   (hierarchical_label "ARR_CURRENT" (shape input) (at 166.37 90.17 0) (fields_autoplaced)
     (effects (font (size 1.27 1.27)) (justify left))
@@
     )
   )
+  (symbol (lib_id "power:PWR_FLAG") (at 170.18 80.01 0) (unit 1)
+    (in_bom yes) (on_board yes) (dnp no)
+    (property "Reference" "#FLG0203" (at 170.18 78.105 0)
+      (effects (font (size 1.27 1.27)) hide)
+    )
+    (property "Value" "PWR_FLAG" (at 172.72 81.28 0)
+      (effects (font (size 1.27 1.27)))
+    )
+    (property "Footprint" "" (at 170.18 80.01 0)
+      (effects (font (size 1.27 1.27)) hide)
+    )
+    (property "Datasheet" "~" (at 170.18 80.01 0)
+      (effects (font (size 1.27 1.27)) hide)
+    )
+    (pin "1")
+    (instances
+      (project "mppt"
+        (path "/06fd3a42-664d-41bc-bf0f-b5ee0ddcc902/90f57858-b3ac-468b-8edb-acb0ab266950"
+          (reference "#FLG0203") (unit 1)
+        )
+      )
+    )
+  )
   (symbol (lib_id "Connector:TestPoint") (at 182.88 105.41 0) (unit 1)
     (in_bom yes) (on_board yes) (dnp no) (fields_autoplaced)
-    (property "Reference" "TP201" (at 185.42 101.473 0)
+    (property "Reference" "TP202" (at 185.42 101.473 0)
       (effects (font (size 1.27 1.27)) (justify left))
     )
@@
       (project "mppt"
         (path "/06fd3a42-664d-41bc-bf0f-b5ee0ddcc902/90f57858-b3ac-468b-8edb-acb0ab266950"
-          (reference "TP201") (unit 1)
+          (reference "TP202") (unit 1)
         )
       )
@@
   (symbol (lib_id "Device:LED") (at 93.98 96.52 90) (unit 1)
     (in_bom yes) (on_board yes) (dnp no) (fields_autoplaced)
-    (property "Reference" "D203" (at 97.79 97.4725 90)
+    (property "Reference" "D202" (at 97.79 97.4725 90)
       (effects (font (size 1.27 1.27)) (justify right))
     )
@@
       (project "mppt"
         (path "/06fd3a42-664d-41bc-bf0f-b5ee0ddcc902/90f57858-b3ac-468b-8edb-acb0ab266950"
-          (reference "D203") (unit 1)
+          (reference "D202") (unit 1)
         )
       )
@@
   (symbol (lib_id "Connector:TestPoint") (at 175.26 80.01 270) (unit 1)
     (in_bom yes) (on_board yes) (dnp no) (fields_autoplaced)
-    (property "Reference" "TP203" (at 180.34 79.375 90)
+    (property "Reference" "TP201" (at 180.34 79.375 90)
       (effects (font (size 1.27 1.27)) (justify left))
     )
@@
       (project "mppt"
         (path "/06fd3a42-664d-41bc-bf0f-b5ee0ddcc902/90f57858-b3ac-468b-8edb-acb0ab266950"
-          (reference "TP203") (unit 1)
+          (reference "TP201") (unit 1)
         )
       )
@@
   (symbol (lib_id "Device:LED") (at 82.55 96.52 90) (unit 1)
     (in_bom yes) (on_board yes) (dnp no) (fields_autoplaced)
-    (property "Reference" "D204" (at 86.36 97.4725 90)
+    (property "Reference" "D201" (at 86.36 97.4725 90)
       (effects (font (size 1.27 1.27)) (justify right))
     )
@@
       (project "mppt"
         (path "/06fd3a42-664d-41bc-bf0f-b5ee0ddcc902/90f57858-b3ac-468b-8edb-acb0ab266950"
-          (reference "D204") (unit 1)
+          (reference "D201") (unit 1)
         )
       )
@@
   (symbol (lib_id "Device:LED") (at 105.41 96.52 90) (unit 1)
     (in_bom yes) (on_board yes) (dnp no) (fields_autoplaced)
-    (property "Reference" "D202" (at 109.22 97.4725 90)
+    (property "Reference" "D203" (at 109.22 97.4725 90)
       (effects (font (size 1.27 1.27)) (justify right))
     )
@@
       (project "mppt"
         (path "/06fd3a42-664d-41bc-bf0f-b5ee0ddcc902/90f57858-b3ac-468b-8edb-acb0ab266950"
-          (reference "D202") (unit 1)
+          (reference "D203") (unit 1)
         )
       )
@@
   (symbol (lib_id "Connector:TestPoint") (at 190.5 72.39 0) (unit 1)
     (in_bom yes) (on_board yes) (dnp no) (fields_autoplaced)
-    (property "Reference" "TP202" (at 193.04 68.453 0)
+    (property "Reference" "TP203" (at 193.04 68.453 0)
       (effects (font (size 1.27 1.27)) (justify left))
     )
@@
       (project "mppt"
         (path "/06fd3a42-664d-41bc-bf0f-b5ee0ddcc902/90f57858-b3ac-468b-8edb-acb0ab266950"
-          (reference "TP202") (unit 1)
-        )
-      )
+          (reference "TP203") (unit 1)
+        )
+      )
