File: hw/controller.kicad_sch (KiCad schematic)
At the start: 14 parts, among them J201 1935776, SW201 SW_Push, U201 MCU_Nucleo_L432KC

Commit message: Added proper signal TPs for Vsw, both gate signals, and PWM, added BNC connector for PWM control signal to STM analog pin, increased Vsw zone on F.cu, in.1, and in.2, reduced vias directly under fets, changed heatsink holesto pads for proper zone margins
Parts:
- added J1: BNC, mppt:CONBNC002, symbol CONBNC002:CONBNC002
- added TP301: PWM Test Point, mppt:SignalTP, symbol Connector:TestPoint_2Pole
Connections:
- net GND: now also J1.1, TP301.2
- net PWM: now also TP301.1
- net PWM_ctrl: now reaches U201.19 (A0)
- net PWM_ctrl: now also J1.2
- no-connect marks 14 -> 15
Changed lines of the file:
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@@
   (junction (at 175.26 80.01) (diameter 0) (color 0 0 0 0)
   )
+  (junction (at 195.58 78.74) (diameter 0) (color 0 0 0 0)
+  )
   (junction (at 184.15 77.47) (diameter 0) (color 0 0 0 0)
+  )
+  (junction (at 195.58 97.79) (diameter 0) (color 0 0 0 0)
   )
   (junction (at 190.5 78.74) (diameter 0) (color 0 0 0 0)
@@
   (no_connect (at 140.97 92.71))
   (no_connect (at 140.97 105.41))
+  (no_connect (at 218.44 100.33))
+  (no_connect (at 218.44 97.79))
   (no_connect (at 140.97 95.25))
   (no_connect (at 140.97 100.33))
@@
   (no_connect (at 140.97 85.09))
   (no_connect (at 140.97 87.63))
-  (no_connect (at 166.37 100.33))
   (no_connect (at 166.37 102.87))
   (wire (pts (xy 93.98 83.82) (xy 93.98 85.09))
@@
     (stroke (width 0) (type default))
   )
-  (wire (pts (xy 190.5 78.74) (xy 199.39 78.74))
+  (wire (pts (xy 190.5 78.74) (xy 195.58 78.74))
+    (stroke (width 0) (type default))
+  )
+  (wire (pts (xy 195.58 97.79) (xy 195.58 78.74))
+    (stroke (width 0) (type default))
+  )
+  (wire (pts (xy 166.37 100.33) (xy 195.58 100.33))
     (stroke (width 0) (type default))
   )
@@
     (stroke (width 0) (type default))
   )
+  (wire (pts (xy 166.37 97.79) (xy 182.88 97.79))
+    (stroke (width 0) (type default))
+  )
   (wire (pts (xy 166.37 105.41) (xy 177.8 105.41))
     (stroke (width 0) (type default))
@@
     (stroke (width 0) (type default))
   )
+  (wire (pts (xy 195.58 78.74) (xy 199.39 78.74))
+    (stroke (width 0) (type default))
+  )
   (wire (pts (xy 130.81 82.55) (xy 140.97 82.55))
     (stroke (width 0) (type default))
@@
     (stroke (width 0) (type default))
   )
+  (wire (pts (xy 193.04 97.79) (xy 195.58 97.79))
+    (stroke (width 0) (type default))
+  )
   (wire (pts (xy 166.37 72.39) (xy 175.26 72.39))
     (stroke (width 0) (type default))
@@
   )
   (label "Tracking" (at 130.81 74.93 0) (fields_autoplaced)
+    (effects (font (size 1.27 1.27)) (justify left bottom))
+  )
+  (label "PWM_ctrl" (at 173.99 100.33 0) (fields_autoplaced)
     (effects (font (size 1.27 1.27)) (justify left bottom))
   )
@@
     )
   )
+  (symbol (lib_id "CONBNC002:CONBNC002") (at 195.58 97.79 0) (unit 1)
+    (in_bom yes) (on_board yes) (dnp no) (fields_autoplaced)
+    (property "Reference" "J1" (at 207.01 90.805 0)
+      (effects (font (size 1.27 1.27)))
+    )
+    (property "Value" "BNC" (at 207.01 93.345 0)
+      (effects (font (size 1.27 1.27)))
+    )
+    (property "Footprint" "mppt:CONBNC002" (at 214.63 95.25 0)
+      (effects (font (size 1.27 1.27)) (justify left) hide)
+    )
+    (property "Datasheet" "" (at 214.63 97.79 0)
+      (effects (font (size 1.27 1.27)) (justify left) hide)
+    )
+    (property "Description" "" (at 214.63 100.33 0)
+      (effects (font (size 1.27 1.27)) (justify left) hide)
+    )
+    (property "Height" "" (at 214.63 102.87 0)
+      (effects (font (size 1.27 1.27)) (justify left) hide)
+    )
+    (property "Mouser Part Number" "" (at 214.63 105.41 0)
+      (effects (font (size 1.27 1.27)) (justify left) hide)
+    )
+    (property "Mouser Price/Stock" "" (at 214.63 107.95 0)
+      (effects (font (size 1.27 1.27)) (justify left) hide)
+    )
+    (property "Manufacturer_Name" "" (at 214.63 110.49 0)
+      (effects (font (size 1.27 1.27)) (justify left) hide)
+    )
+    (property "Manufacturer_Part_Number" "RF1-01A-D-00-75-M" (at 214.63 113.03 0)
+      (effects (font (size 1.27 1.27)) (justify left) hide)
+    )
+    (pin "1")
+    (pin "2")
+    (pin "MH1")
+    (pin "MH2")
+    (instances
+      (project "mppt"
+        (path "/06fd3a42-664d-41bc-bf0f-b5ee0ddcc902/90f57858-b3ac-468b-8edb-acb0ab266950"
+          (reference "J1") (unit 1)
+        )
+      )
+    )
+  )
   (symbol (lib_id "power:GND") (at 93.98 100.33 0) (unit 1)
     (in_bom yes) (on_board yes) (dnp no) (fields_autoplaced)
@@
         )
       )
+    )
+  )
+  (symbol (lib_id "Connector:TestPoint_2Pole") (at 187.96 97.79 0) (unit 1)
+    (in_bom yes) (on_board yes) (dnp no) (fields_autoplaced)
+    (property "Reference" "TP301" (at 187.96 92.71 0)
+      (effects (font (size 1.27 1.27)))
+    )
+    (property "Value" "PWM Test Point" (at 187.96 95.25 0)
+      (effects (font (size 1.27 1.27)))
+    )
+    (property "Footprint" "mppt:SignalTP" (at 187.96 97.79 0)
+      (effects (font (size 1.27 1.27)) hide)
+    )
+    (property "Datasheet" "~" (at 187.96 97.79 0)
+      (effects (font (size 1.27 1.27)) hide)
+    )
+    (pin "1")
+    (pin "2")
+    (instances
+      (project "mppt"
+        (path "/06fd3a42-664d-41bc-bf0f-b5ee0ddcc902/9cd55a57-0ec8-481d-b571-b5fdbe353ce7"
+          (reference "TP301") (unit 1)
+        )
+        (path "/06fd3a42-664d-41bc-bf0f-b5ee0ddcc902/90f57858-b3ac-468b-8edb-acb0ab266950"
+          (reference "TP205") (unit 1)
+        )
+      )

Commit message: changed low-speed test points to through-hole standoffs, created a thermal sink area for high-side fet on B.Cu, and changed some thermal resistors to larger 1225 package where available due to lower cost and better thermal resistance
Parts:
- TP201, TP202, TP203, TP204: footprint TestPoint:TestPoint_Pad_2.0x2.0mm -> TestPoint:TestPoint_Keystone_5000-5004_Miniature
Changed lines of the file:
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@@
       (effects (font (size 1.27 1.27)) (justify left))
     )
-    (property "Footprint" "TestPoint:TestPoint_Pad_2.0x2.0mm" (at 187.96 105.41 0)
+    (property "Footprint" "TestPoint:TestPoint_Keystone_5000-5004_Miniature" (at 187.96 105.41 0)
       (effects (font (size 1.27 1.27)) hide)
     )
@@
       (effects (font (size 1.27 1.27)) (justify right))
     )
-    (property "Footprint" "TestPoint:TestPoint_Pad_2.0x2.0mm" (at 194.31 78.74 0)
+    (property "Footprint" "TestPoint:TestPoint_Keystone_5000-5004_Miniature" (at 194.31 78.74 0)
       (effects (font (size 1.27 1.27)) hide)
     )
@@
       (effects (font (size 1.27 1.27)) (justify left))
     )
-    (property "Footprint" "TestPoint:TestPoint_Pad_2.0x2.0mm" (at 175.26 85.09 0)
+    (property "Footprint" "TestPoint:TestPoint_Keystone_5000-5004_Miniature" (at 175.26 85.09 0)
       (effects (font (size 1.27 1.27)) hide)
     )
@@
       (effects (font (size 1.27 1.27)) (justify left))
     )
-    (property "Footprint" "TestPoint:TestPoint_Pad_2.0x2.0mm" (at 195.58 72.39 0)
-      (effects (font (size 1.27 1.27)) hide)
-    )
+    (property "Footprint" "TestPoint:TestPoint_Keystone_5000-5004_Miniature" (at 195.58 72.39 0)
+      (effects (font (size 1.27 1.27)) hide)
+    )
