File: hw/controller.kicad_sch (KiCad schematic)
At the start: 15 parts, among them J201 1935776, J202 BNC, SW201 SW_Push, U201 MCU_Nucleo_L432KC

Commit message: v0.2.0
Parts:
- removed J201: 1935776, footprints:1935776, symbol 1935776:1935776
- removed J202: BNC, footprints:CONBNC002, symbol CONBNC002:CONBNC002
- removed SW201: SW_Push, footprints:TS046643BK100SMT, symbol TS04-66-43-BK-100-SMT:TS04-66-43-BK-100-SMT
- removed TP204: TestPoint_2Pole, footprints:SignalTP, symbol Connector:TestPoint_2Pole
- removed TP205: GND MCU TP, TestPoint:TestPoint_Keystone_5000-5004_Miniature, symbol Connector:TestPoint
- removed U201: MCU_Nucleo_L432KC, footprints:MODULE_NUCLEO-L432KC, symbol MPPT:MCU_Nucleo_L432KC
- added D204, D205: BLUE, LED_SMD:LED_0603_1608Metric, symbol Device:LED
- added J201: 43650-0227, footprints:molex_microfit_43650_0227, symbol molex_microfit_43650_0227:43650-0227
- added R203, R204, R205: 100, Resistor_SMD:R_0402_1005Metric, symbol Device:R
- added S201: TS-1187A-B-A-B, footprints:xkb_TS_1187A_B_A_B, symbol xkb_TS_1187A_B_A_B:TS-1187A-B-A-B
- added TP204: 12V TP, TestPoint:TestPoint_Pad_1.0x1.0mm, symbol Connector:TestPoint
- added U201: NUCLEO-L432KC, footprints:stm_nucleo_L432KC, symbol stm_nucleo_L432KC:NUCLEO-L432KC
- D201: value RED -> YELLOW; footprint LED_SMD:LED_0402_1005Metric -> LED_SMD:LED_0603_1608Metric; Cost 0.43 -> 0.0206; Distributor Mouser -> JLCPCB; LCSC Part # (none) -> C72038; Manufacturer Kingbright -> Everlight Elec; P/N 604-APHHS1005SURCK -> 19-213/Y2C-CQ2R2L/3T(CY)
- D202: value YELLOW -> GREEN; footprint LED_SMD:LED_0402_1005Metric -> LED_SMD:LED_0603_1608Metric; Cost 0.34 -> 0.0248; Distributor Mouser -> JLCPCB; LCSC Part # (none) -> C72043; Manufacturer Kingbright -> Everlight Elec; P/N 604-APHHS1005SYCK -> 19-217/GHC-YR1S2/3T
- D203: value BLUE -> GREEN; footprint LED_SMD:LED_0402_1005Metric -> LED_SMD:LED_0603_1608Metric; Cost 0.37 -> 0.0248; Distributor Mouser -> JLCPCB; LCSC Part # (none) -> C72043; Manufacturer Kingbright -> Everlight Elec; P/N 604-APHHS1005QBCD -> 19-217/GHC-YR1S2/3T
- R201, R202: Cost 0.0005 -> 0.0004
- TP201: value 5V TP -> 3V3 TP; footprint TestPoint:TestPoint_Keystone_5000-5004_Miniature -> TestPoint:TestPoint_Pad_1.0x1.0mm; Color Red -> (none); Cost 0.36 -> (none); Distributor Mouser -> (none); Manufacturer Keystone Electronics -> (none); P/N 534-5000 -> (none)
- TP202: value 3.3V TP -> 5V TP; footprint TestPoint:TestPoint_Keystone_5000-5004_Miniature -> TestPoint:TestPoint_Pad_1.0x1.0mm; Color Red -> (none); Cost 0.36 -> (none); Distributor Mouser -> (none); Manufacturer Keystone Electronics -> (none); P/N 534-5000 -> (none)
- TP203: value 12V TP -> GND TP; footprint TestPoint:TestPoint_Keystone_5000-5004_Miniature -> TestPoint:TestPoint_Pad_1.0x1.0mm; Color Red -> (none); Cost 0.36 -> (none); Distributor Mouser -> (none); Manufacturer Keystone Electronics -> (none); P/N 534-5000 -> (none)
Connections:
- net +3.3V is gone; now on net +5V: TP202.1
- net +12V: now also J201.1, TP204.1, U201.30 (VIN); no longer TP203.1
- net +5V: now also U201.27 (+5V); no longer TP201.1
- net ARR_I: now also U201.19 (A0)
- net ARR_V: now also U201.20 (A1)
- net BATT_I: now also U201.26 (A7)
- net BATT_V: now also U201.25 (A6)
- net Error: now also U201.6 (D3)
- net GND: now also TP203.1, D204.1 (K), D205.1 (K), J201.2, S201.C, S201.D, U201.29 (GND), U201.4 (GND)
- net Heartbeat: now also R203.2, U201.1 (D1); no longer D203.2 (A)
- net PWM: now also U201.24 (A5)
- net PWM_EN: now also U201.23 (A4)
- net Reset: now also S201.A, S201.B, U201.28 (RST), U201.3 (RST)
- net Tracking: now also U201.2 (D0)
- new net: D203.2 (A), R203.1
- new net: D205.2 (A), R205.1
- new net: D204.2 (A), R204.1
- new net +3V3: TP201.1, U201.17 (+3V3)
- new net CAN_RX: R205.2, U201.13 (D10)
- new net CAN_TX: R204.2, U201.5 (D2)
- no-connect marks 13 -> 12
Other:
- note added: "Controller"
- note added: "LEDs"
- note added: "SCL"
- note added: "SDA"
- note added: "Testpoints"
- note removed: "I2C1_SCL"
- note removed: "I2C1_SDA"
- note removed: "USB_DM|CAN1_RD"
- note removed: "USB_DP|CAN1_TD"
- company: UT LHR Solar -> LHR Solar
