File: hw/sensors.kicad_sch (KiCad schematic)
At the start: 29 parts, among them J201 BNC, U401 OPA990, U402 INA210, U403 OPA990, U404 INA210

Commit message: savestate layout
Parts:
- removed TP401: +ARR, TestPoint:TestPoint_Keystone_5000-5004_Miniature, symbol Connector:TestPoint
- removed TP406: +BATT, TestPoint:TestPoint_Keystone_5000-5004_Miniature, symbol Connector:TestPoint
- added TP401, TP410: TestPoint_2Pole, mppt:SignalTP, symbol Connector:TestPoint_2Pole
- R403, R406: P/N (none) -> 755-PMR18EZPFV2L00
- renumbered TP407 to TP406, TP408 to TP407, TP409 to TP408, TP410 to TP409
Connections:
- net +ARR: now also TP401.1
- net +BATT: now also TP410.1
- net GND: now also J201.MH1, J201.MH2, TP401.2, TP410.2
- no-connect marks 2 -> 0
Other:
- moved on the sheet: J201
