File: hw/sensors.kicad_sch (KiCad schematic)
At the start: 30 parts, among them IC401 INA210CQDCKRQ1, IC402 OPA990IDCKR, IC403 OPA990IDCKR, IC404 INA210CQDCKRQ1

Commit message: v3 savestate
Parts:
- added TH? (x3): PT100, symbol Sensor_Temperature:PT100
Other:
- note added: "RTD Sensors"
- moved on the sheet: C401, C402, C403, C404, D401, D402, D403, D404, IC401, IC402, IC403, IC404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

Commit message: savestate
Parts:
- removed TH? (x3): PT100, symbol Sensor_Temperature:PT100
Other:
- added sheet rtd_sensor_0 (rtd_sensor.kicad_sch)
- added sheet rtd_sensor_1 (rtd_sensor.kicad_sch)
- added sheet rtd_sensor_2 (rtd_sensor.kicad_sch)
- note added: "For a maximum of 8, we tie SPI MOSI/MISO/SCLK/DRDY for all of them and use the CS pin for controlling which ones get to send across data on the bus."
