File: hw/sensors.kicad_sch (KiCad schematic)
At the start: 30 parts, among them IC401 INA210CQDCKRQ1, IC402 OPA990IDCKR, IC403 OPA990IDCKR, IC404 INA210CQDCKRQ1

Commit message: bugfix for wrong adc pin for batt current measurements
Parts:
- C401, C402, C403, C404: Cost 0.0068 -> 0.0063; LCSC Part # C307331 -> CL05B104KB54PNC; Notes (none) -> Rated for 50V.
- IC401, IC404: Cost 1.52 -> 1.020; Distributor Mouser -> Texas Instruments
- IC402, IC403: Cost 1.19 -> 0.865; Distributor Mouser -> Texas Instruments
Changed lines of the file:
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@@
       (effects (font (size 1 1)) (justify left top) hide)
     )
-    (property "Distributor" "Mouser" (at 104.14 111.76 0)
+    (property "Distributor" "Texas Instruments" (at 104.14 111.76 0)
       (effects (font (size 1 1)) hide)
     )
@@
       (effects (font (size 1 1)) hide)
     )
-    (property "Cost" "1.52" (at 104.14 110.49 0)
+    (property "Cost" "1.020" (at 104.14 110.49 0)
       (effects (font (size 1 1)) hide)
     )
@@
       (effects (font (size 1 1)) (justify left) hide)
     )
-    (property "Datasheet" "https://datasheet.lcsc.com/lcsc/1810191222_Samsung-Electro-Mechanics-CL05B104KB54PNC_C307331.pdf" (at 116.84 55.88 0)
+    (property "Datasheet" "https://datasheet.lcsc.com/lcsc/2304140030_Samsung-Electro-Mechanics-CL05B104KB54PNC_C307331.pdf" (at 116.84 55.88 0)
       (effects (font (size 1 1)) (justify left) hide)
     )
@@
       (effects (font (size 1 1)) hide)
     )
-    (property "LCSC Part #" "C307331" (at 125.73 57.15 0)
-      (effects (font (size 1 1)) hide)
-    )
-    (property "Cost" "0.0068" (at 125.73 57.15 0)
-      (effects (font (size 1 1)) hide)
+    (property "LCSC Part #" "CL05B104KB54PNC" (at 125.73 57.15 0)
+      (effects (font (size 1 1)) hide)
+    )
+    (property "Cost" "0.0063" (at 125.73 57.15 0)
+      (effects (font (size 1 1)) hide)
+    )
+    (property "Notes" "Rated for 50V." (at 125.73 57.15 0)
+      (effects (font (size 1.27 1.27)) hide)
     )
     (pin "1")
@@
       (effects (font (size 1 1)) (justify left) hide)
     )
-    (property "Datasheet" "https://datasheet.lcsc.com/lcsc/1810191222_Samsung-Electro-Mechanics-CL05B104KB54PNC_C307331.pdf" (at 184.15 101.6 0)
+    (property "Datasheet" "https://datasheet.lcsc.com/lcsc/2304140030_Samsung-Electro-Mechanics-CL05B104KB54PNC_C307331.pdf" (at 184.15 101.6 0)
       (effects (font (size 1 1)) (justify left) hide)
     )
@@
       (effects (font (size 1 1)) hide)
     )
-    (property "LCSC Part #" "C307331" (at 193.04 102.87 0)
-      (effects (font (size 1 1)) hide)
-    )
-    (property "Cost" "0.0068" (at 193.04 102.87 0)
-      (effects (font (size 1 1)) hide)
+    (property "LCSC Part #" "CL05B104KB54PNC" (at 193.04 102.87 0)
+      (effects (font (size 1 1)) hide)
+    )
+    (property "Cost" "0.0063" (at 193.04 102.87 0)
+      (effects (font (size 1 1)) hide)
+    )
+    (property "Notes" "Rated for 50V." (at 193.04 102.87 0)
+      (effects (font (size 1.27 1.27)) hide)
     )
     (pin "1")
@@
       (effects (font (size 1 1)) (justify left top) hide)
     )
-    (property "Distributor" "Mouser" (at 107.95 67.31 0)
+    (property "Distributor" "Texas Instruments" (at 107.95 67.31 0)
       (effects (font (size 1 1)) hide)
     )
@@
       (effects (font (size 1 1)) hide)
     )
-    (property "Cost" "1.19" (at 107.95 64.77 0)
+    (property "Cost" "0.865" (at 107.95 64.77 0)
       (effects (font (size 1 1)) hide)
     )
@@
       (effects (font (size 1 1)) (justify left top) hide)
     )
-    (property "Distributor" "Mouser" (at 175.26 67.31 0)
+    (property "Distributor" "Texas Instruments" (at 175.26 67.31 0)
       (effects (font (size 1 1)) hide)
     )
@@
       (effects (font (size 1 1)) hide)
     )
-    (property "Cost" "1.19" (at 175.26 64.77 0)
+    (property "Cost" "0.865" (at 175.26 64.77 0)
       (effects (font (size 1 1)) hide)
     )
@@
       (effects (font (size 1 1)) (justify left top) hide)
     )
-    (property "Distributor" "Mouser" (at 175.26 111.76 0)
+    (property "Distributor" "Texas Instruments" (at 175.26 111.76 0)
       (effects (font (size 1 1)) hide)
     )
@@
       (effects (font (size 1 1)) hide)
     )
-    (property "Cost" "1.52" (at 175.26 110.49 0)
+    (property "Cost" "1.020" (at 175.26 110.49 0)
       (effects (font (size 1 1)) hide)
     )
@@
       (effects (font (size 1 1)) (justify left) hide)
     )
-    (property "Datasheet" "https://datasheet.lcsc.com/lcsc/1810191222_Samsung-Electro-Mechanics-CL05B104KB54PNC_C307331.pdf" (at 113.03 101.6 0)
+    (property "Datasheet" "https://datasheet.lcsc.com/lcsc/2304140030_Samsung-Electro-Mechanics-CL05B104KB54PNC_C307331.pdf" (at 113.03 101.6 0)
       (effects (font (size 1 1)) (justify left) hide)
     )
@@
       (effects (font (size 1 1)) hide)
     )
-    (property "LCSC Part #" "C307331" (at 121.92 102.87 0)
-      (effects (font (size 1 1)) hide)
-    )
-    (property "Cost" "0.0068" (at 121.92 102.87 0)
-      (effects (font (size 1 1)) hide)
+    (property "LCSC Part #" "CL05B104KB54PNC" (at 121.92 102.87 0)
+      (effects (font (size 1 1)) hide)
+    )
+    (property "Cost" "0.0063" (at 121.92 102.87 0)
+      (effects (font (size 1 1)) hide)
+    )
+    (property "Notes" "Rated for 50V." (at 121.92 102.87 0)
+      (effects (font (size 1.27 1.27)) hide)
     )
     (pin "1")
@@
       (effects (font (size 1 1)) (justify left) hide)
     )
-    (property "Datasheet" "https://datasheet.lcsc.com/lcsc/1810191222_Samsung-Electro-Mechanics-CL05B104KB54PNC_C307331.pdf" (at 184.15 55.88 0)
+    (property "Datasheet" "https://datasheet.lcsc.com/lcsc/2304140030_Samsung-Electro-Mechanics-CL05B104KB54PNC_C307331.pdf" (at 184.15 55.88 0)
       (effects (font (size 1 1)) (justify left) hide)
     )
@@
       (effects (font (size 1 1)) hide)
     )
-    (property "LCSC Part #" "C307331" (at 193.04 57.15 0)
-      (effects (font (size 1 1)) hide)
-    )
-    (property "Cost" "0.0068" (at 193.04 57.15 0)
-      (effects (font (size 1 1)) hide)
-    )
-    (pin "1")
+    (property "LCSC Part #" "CL05B104KB54PNC" (at 193.04 57.15 0)
+      (effects (font (size 1 1)) hide)
+    )
+    (property "Cost" "0.0063" (at 193.04 57.15 0)
+      (effects (font (size 1 1)) hide)
+    )
+    (property "Notes" "Rated for 50V." (at 193.04 57.15 0)
+      (effects (font (size 1.27 1.27)) hide)
+    )
+    (pin "1")

Commit message: init sch changes
Parts:
- removed C401, C402, C403, C404: 100nF, Capacitor_SMD:C_0402_1005Metric, symbol Device:C_Small
- removed D401, D404: 3.3V Zener, Diode_SMD:D_MiniMELF, symbol Device:D_Zener_Small
- removed D402, D403: 3V3, Diode_SMD:D_MiniMELF, symbol Device:D_Zener_Small
- removed IC401, IC404: INA210CQDCKRQ1, footprints:ti_INA210CQDCKRQ1, symbol ti_INA210CQDCKRQ1:INA210CQDCKRQ1
- removed IC402, IC403: OPA990IDCKR, footprints:ti_OPA990IDCKR, symbol ti_OPA990IDCKR:OPA990IDCKR
- removed R401, R404: 100k, Resistor_SMD:R_0805_2012Metric, symbol Device:R
- removed R402: 3k, Resistor_SMD:R_0805_2012Metric, symbol Device:R
- removed R403, R406: 2m, Resistor_SMD:R_1206_3216Metric, symbol Device:R
- removed R405: 2k, Resistor_SMD:R_0805_2012Metric, symbol Device:R
- removed TP401: +ARR_TP, TestPoint:TestPoint_Pad_1.0x1.0mm, symbol Connector:TestPoint
- removed TP402, TP403, TP408, TP410: GND_TP, TestPoint:TestPoint_Pad_1.0x1.0mm, symbol Connector:TestPoint
- removed TP404: -ARR_TP, TestPoint:TestPoint_Pad_1.0x1.0mm, symbol Connector:TestPoint
- removed TP405: ARRI_TP, TestPoint:TestPoint_Pad_1.0x1.0mm, symbol Connector:TestPoint
- removed TP406: ARRV_TP, TestPoint:TestPoint_Pad_1.0x1.0mm, symbol Connector:TestPoint
- removed TP407: +BATT_TP, TestPoint:TestPoint_Pad_1.0x1.0mm, symbol Connector:TestPoint
- removed TP409: -BATT_TP, TestPoint:TestPoint_Pad_1.0x1.0mm, symbol Connector:TestPoint
- removed TP411: BATTV_TP, TestPoint:TestPoint_Pad_1.0x1.0mm, symbol Connector:TestPoint
- removed TP412: BATTI_TP, TestPoint:TestPoint_Pad_1.0x1.0mm, symbol Connector:TestPoint
- added C17, C20, C22, C23, C26: 100nF, symbol Device:C_Small
- added C21, C27: 1uF, symbol Device:C_Small
- added D2, D4, D6, D7: 3V3, Diode_SMD:D_MiniMELF, symbol Device:D_Zener_Small
- added IC, IC5: OPA990IDCKR, footprints:ti_OPA990IDCKR, symbol ti_OPA990IDCKR:OPA990IDCKR
- added IC2, IC6: INA215CQDCKRQ1, footprints:ti_INA215CQDCKRQ1, symbol ti_INA215CQDCKRQ1:INA215CQDCKRQ1
- added R10: 2.2k, symbol Device:R_Small
- added R11, R6: 2m, symbol Device:R_Small
- added R13, R14, R7, R8: 10k, symbol Device:R_Small
- added R2: 400, symbol Device:R_Small
- added R4, R9: 100k, symbol Device:R_Small
- added R5: 3.3k, symbol Device:R_Small
- added TH1, TH2, TH3, TH4: PT100, symbol Sensor_Temperature:PT100
- added TP15: I_{ARR_REF}, symbol Connector:TestPoint
- added TP16: I_{ARR}, symbol Connector:TestPoint
- added TP17: I_{BATT_REF}, symbol Connector:TestPoint
- added TP18: I_{BATT}, symbol Connector:TestPoint
- added TP4: V_{ARR}, symbol Connector:TestPoint
- added TP5: V_{BATT}, symbol Connector:TestPoint
- added TP6, TP7: GND, symbol Connector:TestPoint
- added U5: MAX31865xTP, Package_DFN_QFN:TQFN-20-1EP_5x5mm_P0.65mm_EP3.25x3.25mm, symbol Sensor_Temperature:MAX31865xTP
- added U6: ADG734, Package_SO:TSSOP-20_4.4x6.5mm_P0.65mm, symbol Analog_Switch:ADG734
Connections:
- net GND: now also C17.2, C20.2, C21.2, C22.2, C26.2, C27.2, D2.2 (A), D4.2 (A), D6.2 (A), D7.2 (A), IC.2 (V-), IC2.2 (GND), IC5.2 (V-), IC6.2 (GND), R10.2, R14.2, R5.2, R8.2, TP6.1, TP7.1, U5.10 (GND), U5.15 (DGND), U5.16 (GND), U5.21 (GND), U5.6 (FORCE2), U6.5 (VSS), U6.6 (GND)
- new net: TH1.1, U6.2
- new net: IC5.1 (IN+), R10.1, R9.2
- new net: R2.1, U5.1 (BIAS), U5.2 (REFIN+)
- new net: R2.2, U5.3 (REFIN-), U5.4 (ISENSOR)
- new net: IC.1 (IN+), R4.2, R5.1
- new net: TH4.1, U6.19
- new net: TH3.1, U6.12
- new net: TH2.1, U6.9
- new net +3V3: C17.1, C20.1, C21.1, C22.1, C26.1, C27.1, IC.5 (V+), IC2.3 (V+), IC5.5 (V+), IC6.3 (V+), R13.1, R7.1, U5.19 (DVDD), U5.20 (VDD), U6.16 (VDD)
- new net I_{ARR_REF}: IC2.1 (REF), R7.2, R8.1, TP15.1
- new net I_{ARR}: D2.1 (K), IC2.6 (OUT), TP16.1
- new net I_{BATT_REF}: IC6.1 (REF), R13.2, R14.1, TP17.1
- new net I_{BATT}: D6.1 (K), IC6.6 (OUT), TP18.1
- new net RTD_GATE: U6.10
- new net RTD_IND: U6.1
- new net RTD_SCLK: U5.12 (SCLK)
- new net RTD_SDI: U5.11 (SDI)
- new net RTD_SDO: U5.14 (SDO)
- new net RTD_SINK: C23.2, TH1.2, TH2.2, TH3.2, TH4.2, U5.8 (RTDIN-), U5.9 (FORCE-)
- new net RTD_SOURCE: C23.1, U5.5 (FORCE+), U5.7 (RTDIN+), U6.13, U6.18, U6.3, U6.8
- new net RTD_SWH: U6.20
- new net RTD_SWL: U6.11
- new net V_{ARR+}: IC2.4 (IN+), R4.1, R6.1
- new net V_{ARR}: D4.1 (K), IC.3 (IN-), IC.4 (OUT), TP4.1
- new net V_{BATT+}: IC6.4 (IN+), R11.1, R9.1
- new net V_{BATT}: D7.1 (K), IC5.3 (IN-), IC5.4 (OUT), TP5.1
- new net V_{DCI+}: IC2.5 (IN-), R6.2
- new net V_{DCO+}: IC6.5 (IN-), R11.2
- new net ~{RTD_CS}: U5.13 (~{CS})
- new net ~{RTD_DRDY}: U5.18 (~{DRDY})
- no-connect marks 0 -> 4
Other:
- note added: "-9A to 9A"
- note added: "2.5 Ohm R_{ON} 6.4 deg C drift correction required"
- note added: "Gate Driver"
- note added: "High Side Switch"
- note added: "High precision"
- note added: "Inductor"
- note added: "Low Side Switch"
- note added: "Measure REF to cancel ext impedance"
- note added: "Oversized to reduce VREF noise"
- note added: "Per V_{DD}"
- note added: "Temperature Sensor"
- note removed: "0-113V"
- note removed: "0-168V"
- note removed: "0-3.3V"
- note removed: "8.25A 0-16.5mV"

Commit message: v0.3.0rc (v1.0.0rc) sch complete
Parts:
- removed C17, C20, C22, C23, C26: 100nF, symbol Device:C_Small
- removed C21, C27: 1uF, symbol Device:C_Small
- removed D2, D4, D6, D7: 3V3, Diode_SMD:D_MiniMELF, symbol Device:D_Zener_Small
- removed IC, IC5: OPA990IDCKR, footprints:ti_OPA990IDCKR, symbol ti_OPA990IDCKR:OPA990IDCKR
- removed IC2, IC6: INA215CQDCKRQ1, footprints:ti_INA215CQDCKRQ1, symbol ti_INA215CQDCKRQ1:INA215CQDCKRQ1
- removed R10: 2.2k, symbol Device:R_Small
- removed R11, R6: 2m, symbol Device:R_Small
- removed R13, R14, R7, R8: 10k, symbol Device:R_Small
- removed R2: 400, symbol Device:R_Small
- removed R4, R9: 100k, symbol Device:R_Small
- removed R5: 3.3k, symbol Device:R_Small
- removed TH1, TH2, TH3, TH4: PT100, symbol Sensor_Temperature:PT100
- removed TP15: I_{ARR_REF}, symbol Connector:TestPoint
- removed TP16: I_{ARR}, symbol Connector:TestPoint
- removed TP17: I_{BATT_REF}, symbol Connector:TestPoint
- removed TP18: I_{BATT}, symbol Connector:TestPoint
- removed TP4: V_{ARR}, symbol Connector:TestPoint
- removed TP5: V_{BATT}, symbol Connector:TestPoint
- removed TP6, TP7: GND, symbol Connector:TestPoint
- removed U5: MAX31865xTP, Package_DFN_QFN:TQFN-20-1EP_5x5mm_P0.65mm_EP3.25x3.25mm, symbol Sensor_Temperature:MAX31865xTP
- removed U6: ADG734, Package_SO:TSSOP-20_4.4x6.5mm_P0.65mm, symbol Analog_Switch:ADG734
- added C401, C402: 100p, Resistor_SMD:R_0402_1005Metric, symbol Device:C_Small
- added C403, C404, C409, C410, C415, C416, C419, C420, C435, C436, C437: 1u, Resistor_SMD:R_0402_1005Metric, symbol Device:C_Small
- added C405, C406, C411, C412, C413, C414, C417, C418, C425, C426, C429, C430, C433, C434: 100n, Resistor_SMD:R_0402_1005Metric, symbol Device:C_Small
- added C407, C408: 10n, Resistor_SMD:R_0402_1005Metric, symbol Device:C_Small
- added C421, C422, C423, C424, C427, C428, C431, C432: 330p, Resistor_SMD:R_0402_1005Metric, symbol Device:C_Small
- added D401, D402, D403, D404: 3.3, Diode_SMD:D_SOD-123, symbol Device:D_Small
- added D405, D406: GRN, LED_SMD:LED_0402_1005Metric, symbol Device:LED_Small
- added R401, R403: 150k, Resistor_SMD:R_0805_2012Metric, symbol Device:R_Small
- added R402, R404: 2.5k, Resistor_SMD:R_0805_2012Metric, symbol Device:R_Small
- added R405, R406: 4mO, Resistor_SMD:R_2512_6332Metric, symbol Device:R_Small
- added R407, R408, R409, R410: 10, Resistor_SMD:R_0402_1005Metric, symbol Device:R_Small
- added R411, R412, R413, R414, R415, R416, R417, R418, R419, R420, R421, R422, R423, R424, R425, R426, R427, R429: 3.3k, Resistor_SMD:R_0402_1005Metric, symbol Device:R_Small
- added R428, R430: 10k, Resistor_SMD:R_0402_1005Metric, symbol Device:R_Small
- added R431, R432: 330, Resistor_SMD:R_0402_1005Metric, symbol Device:R_Small
- added R433: 1k, Resistor_SMD:R_0402_1005Metric, symbol Device:R_Small
- added SB401, SB402: Jumper, Jumper:SolderJumper-2_P1.3mm_Open_TrianglePad1.0x1.5mm, symbol Jumper:SolderJumper_2_Bridged
- added TP401: VBUS_SENSE, TestPoint:TestPoint_Keystone_5000-5004_Miniature, symbol Connector:TestPoint
- added TP402: GND, TestPoint:TestPoint_Keystone_5000-5004_Miniature, symbol Connector:TestPoint
- added TP403: VBUS_SENSE_ISO, TestPoint:TestPoint_Keystone_5000-5004_Miniature, symbol Connector:TestPoint
- added TP404: GNDPWR, TestPoint:TestPoint_Keystone_5000-5004_Miniature, symbol Connector:TestPoint
- added TP405: V_{ARR}, TestPoint:TestPoint_Keystone_5000-5004_Miniature, symbol Connector:TestPoint
- added TP406: I_{ARR}, TestPoint:TestPoint_Keystone_5000-5004_Miniature, symbol Connector:TestPoint
- added TP407: V_{ARR+}, TestPoint:TestPoint_Keystone_5000-5004_Miniature, symbol Connector:TestPoint
- added TP408: V_{ARR-}, TestPoint:TestPoint_Keystone_5000-5004_Miniature, symbol Connector:TestPoint
- added TP409: V_{BAT}, TestPoint:TestPoint_Keystone_5000-5004_Miniature, symbol Connector:TestPoint
- added TP410: I_{BAT}, TestPoint:TestPoint_Keystone_5000-5004_Miniature, symbol Connector:TestPoint
- added TP411: V_{BAT+}, TestPoint:TestPoint_Keystone_5000-5004_Miniature, symbol Connector:TestPoint
- added TP412: V_{BAT-}, TestPoint:TestPoint_Keystone_5000-5004_Miniature, symbol Connector:TestPoint
- added TP413: T_{IND}, TestPoint:TestPoint_Keystone_5000-5004_Miniature, symbol Connector:TestPoint
- added TP414: T_{SWL}, TestPoint:TestPoint_Keystone_5000-5004_Miniature, symbol Connector:TestPoint
- added TP415: T_{SWH}, TestPoint:TestPoint_Keystone_5000-5004_Miniature, symbol Connector:TestPoint
- added TP416: T_{GATE}, TestPoint:TestPoint_Keystone_5000-5004_Miniature, symbol Connector:TestPoint
- added U401, U402: AMC1211, footprints:ti_AMC1211_DWV, symbol ti_AMC1211:AMC1211AQDWVRQ1
- added U403, U404: AMC1202, footprints:ti_AMC1202_DWV, symbol ti_AMC1202:AMC1202DWVR
- added U405, U406, U407, U408, U409, U410: TLV9001, Package_TO_SOT_SMD:SOT-363_SC-70-6, symbol ti_TLV9001:TLV9001
- added U411, U412, U413, U414: MCP9700A, Connector_JST:JST_PH_B3B-PH-K_1x03_P2.00mm_Vertical, symbol Sensor_Temperature:MCP9700Ax-ELT
Connections:
- net GND: now also C413.2, C414.2, C415.2, C416.2, C417.2, C418.2, C419.2, C420.2, C421.2, C422.2, C423.2, C424.2, C425.2, C426.2, C429.2, C430.2, C433.2, C434.2, C435.2, C436.2, D401.2 (A), D402.2 (A), D403.2 (A), D404.2 (A), D405.1 (K), R419.2, R420.2, R423.2, R424.2, R428.2, R430.2, TP402.1, U401.5 (GND2), U402.5 (GND2), U403.5 (GND2), U404.5 (GND2), U405.2 (V-), U405.5 (~{SHDN}), U406.2 (V-), U406.5 (~{SHDN}), U407.2 (V-), U407.5 (~{SHDN}), U408.2 (V-), U408.5 (~{SHDN}), U409.2 (V-), U409.5 (~{SHDN}), U410.2 (V-), U410.5 (~{SHDN}), U411.3 (GND), U412.3 (GND), U413.3 (GND), U414.3 (GND)
- net I_{ARR}: now also C431.2, D403.1 (K), R425.1, TP406.1, U407.4
- net V_{ARR+}: now also R401.1, TP407.1
- net V_{ARR}: now also R427.1, TP405.1, U409.4
- new net: C424.1, R417.1, R424.1, U408.1 (+)
- new net: C432.1, R418.1, R426.2, U408.3 (-)
- new net: C423.1, R415.1, R423.1, U407.1 (+)
- new net: C431.1, R416.1, R425.2, U407.3 (-)
- new net: C428.1, R414.1, R422.2, U406.3 (-)
- new net: R414.2, U402.6 (VOUTN)
- new net: C407.2, R408.1, U403.3 (INN)
- new net: R416.2, U403.6 (OUTN)
- new net: C427.2, D401.1 (K), R421.1, U405.4, U409.1 (+)
- new net: C421.1, R411.1, R419.1, U405.1 (+)
- new net: D406.2 (A), R433.2
- new net: C428.2, D402.1 (K), R422.1, U406.4, U410.1 (+)
- new net: R429.2, R430.1, U410.3 (-)
- new net: C402.1, R403.2, R404.1, U402.2 (VIN)
- new net: C427.1, R412.1, R421.2, U405.3 (-)
- new net: C407.1, R407.2, U403.2 (INP)
- new net: R415.2, U403.7 (OUTP)
- new net: C422.1, R413.1, R420.1, U406.1 (+)
- new net: D405.2 (A), R431.2
- new net: R427.2, R428.1, U409.3 (-)
- new net: C408.2, R410.1, U404.3 (INN)
- new net: C401.1, R401.2, R402.1, U401.2 (VIN)
- new net: R418.2, U404.6 (OUTN)
- new net: C435.1, R432.1, U411.1 (V_{DD}), U412.1 (V_{DD}), U413.1 (V_{DD}), U414.1 (V_{DD})
- new net: R413.2, U402.7 (VOUTP)
- new net: C408.1, R409.2, U404.2 (INP)
- new net: R417.2, U404.7 (OUTP)
- new net: R412.2, U401.6 (VOUTN)
- new net: R411.2, U401.7 (VOUTP)
- new net +3.3VP: SB401.1 (A)
- new net +5VP: SB402.1 (A)
- new net GNDPWR: C401.2, C402.2, C403.2, C404.2, C405.2, C406.2, C409.2, C410.2, C411.2, C412.2, C437.2, D406.1 (K), R402.2, R404.2, R405.2, R406.2, R408.2, R410.2, TP404.1, U401.3 (SHTDN), U401.4 (GND1), U402.3 (SHTDN), U402.4 (GND1), U403.4 (GND1), U404.4 (GND1)
- new net I_{BAT}: C432.2, D404.1 (K), R426.1, TP410.1, U408.4
- new net TEMP_GATE: TP416.1, U412.2 (V_{OUT})
- new net TEMP_IND: TP413.1, U411.2 (V_{OUT})
- new net TEMP_SWH: TP415.1, U413.2 (V_{OUT})
- new net TEMP_SWL: TP414.1, U414.2 (V_{OUT})
- new net VBUS_SENSE: C413.1, C414.1, C415.1, C416.1, C417.1, C418.1, C419.1, C420.1, C425.1, C426.1, C429.1, C430.1, C433.1, C434.1, C436.1, R431.1, R432.2, SB401.2 (B), TP401.1, U401.8 (VDD2), U402.8 (VDD2), U403.8 (VDD2), U404.8 (VDD2), U405.6 (V+), U406.6 (V+), U407.6 (V+), U408.6 (V+), U409.6 (V+), U410.6 (V+)
- new net VBUS_SENSE_ISO: C403.1, C404.1, C405.1, C406.1, C409.1, C410.1, C411.1, C412.1, C437.1, R433.1, SB402.2 (B), TP403.1, U401.1 (VDD1), U402.1 (VDD1), U403.1 (VDD1), U404.1 (VDD1)
- new net V_{ARR-}: R405.1, R407.1, TP408.1
- new net V_{BAT+}: R403.1, TP411.1
- new net V_{BAT-}: R406.1, R409.1, TP412.1
- new net V_{BAT}: R429.1, TP409.1, U410.4
- no-connect marks 4 -> 0
Other:
- note added: "150V 2.5V"
- note added: "400mW * SF diss"
- note added: "Sensors"
- note added: "[0, 2.458]V"
- note added: "[0, 3.274]V"
- note added: "[0, 3.28]V"
- note added: "[0.21, 2.67]V"
- note added: "±10A ±40mV"
- note added: "±2.05V"
- note removed: "-9A to 9A"
- note removed: "2.5 Ohm R_{ON} 6.4 deg C drift correction required"
- note removed: "Array Current Sensor"
- note removed: "Array Voltage Sensor"
- note removed: "Battery Current Sensor"
- note removed: "Battery Voltage Sensor"
- note removed: "Gate Driver"
- note removed: "High Side Switch"
- note removed: "High precision"
- note removed: "Inductor"
- note removed: "Low Side Switch"
- note removed: "Measure REF to cancel ext impedance"
- note removed: "Oversized to reduce VREF noise"
- note removed: "Per V_{DD}"
- note removed: "Temperature Sensor"
