File: hw/mppt.kicad_pcb (KiCad board)
At the start: 4 copper layers, 100 x 55 mm, 74 parts, among them J201 1935776, J202 BNC, J301 1935776, J302 1935776, J401 BNC, Q301 SW_L, Q302 SW_H, SW201 SW_Push, U201 MCU_Nucleo_L432KC, U401 OPA990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

Commit message: final layout
Parts:
- added C304: 18uF, Capacitor_THT:C_Radial_D10.0mm_H16.0mm_P5.00mm, F.Cu at (168.8, 114.0)
- added D301: Schottky, Diode_THT:D_5W_P5.08mm_Vertical_AnodeUp, F.Cu at (148.0, 116.0)
- added R301: R, Resistor_THT:R_Radial_Power_L11.0mm_W7.0mm_P5.00mm, B.Cu at (148.0, 111.0)
- added TJ101: Thermal Jumper, mppt:1225_SMD, F.Cu at (157.8, 107.3)
- added TJ102: Thermal Jumper, mppt:1225_SMD, F.Cu at (144.8, 97.8)
- added TJ103: Thermal Jumper, mppt:1225_SMD, F.Cu at (148.0, 90.0)
- added TP302: TestPoint_2Pole, mppt:SignalTP, F.Cu at (148.8, 95.7)
- C302: value 1uF -> CP; footprint Capacitor_SMD:C_2220_5650Metric -> Capacitor_THT:C_Radial_D10.0mm_H12.5mm_P5.00mm
- C303: value 18uF -> 1uF; footprint Capacitor_THT:C_Radial_D10.0mm_H16.0mm_P5.00mm -> Capacitor_SMD:C_2220_5650Metric; moved to B.Cu
- REF**: moved to F.Cu
- moved REF** 30.3 mm to (127.9, 98.2), turned to 0 degrees
- moved TP301 19.2 mm to (156.5, 112.8), turned to 180 degrees
- moved C301 19.2 mm to (105.0, 117.5), turned to 90 degrees
- moved C303 19.1 mm to (162.2, 98.5)
- moved C302 16.5 mm to (156.5, 114.0), turned to 0 degrees
- moved REF** 5.23 mm to (126.1, 110.7)
- moved L301 3.05 mm to (126.8, 104.7)
- moved TP502 0.42 mm to (153.1, 87.6), turned to 45 degrees
Connections:
- C302 pad 1: /V_BATT+ -> Net-(D301-K)
- TP301 pad 1: /V_SW -> Net-(D301-K)
Routing:
- net Net-(D301-K): track 0.00 -> 9.33 mm
- net /converter/G1: track 15.6 -> 16.6 mm

Commit message: temp for matthew to stitch
Parts:
- added C305: 18uF, Capacitor_THT:C_Radial_D10.0mm_H16.0mm_P5.00mm, F.Cu at (174.7, 114.5)
- added TJ104: Thermal Jumper, Resistor_SMD:R_0805_2012Metric, F.Cu at (172.8, 90.1)
- moved TP406 4.56 mm to (186.4, 110.2)
- moved C304 2.53 mm to (166.8, 112.3)
Connections:
- net Net-(D301-K) renamed /converter/Vsnub
Routing:
- net /converter/V_BATT-: track 15.5 -> 13.9 mm
Changed lines of the file:
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@@
   (net 56 "Net-(U501-LO)")
   (net 57 "Net-(U501-HO)")
-  (net 58 "Net-(D301-K)")
+  (net 58 "/converter/Vsnub")
   (footprint "Symbol:ESD-Logo_8.9x8mm_SilkScreen" (layer "F.Cu")
     (at 127.88 98.22)
@@
   )
   (footprint "Capacitor_THT:C_Radial_D10.0mm_H16.0mm_P5.00mm" (layer "F.Cu")
-    (at 168.75 114)
+    (at 166.85 112.325)
     (descr "C, Radial series, Radial, pin pitch=5.00mm, diameter=10mm, height=16mm, Non-Polar Electrolytic Capacitor")
     (tags "C Radial series Radial pin pitch 5.00mm diameter 10mm height 16mm Non-Polar Electrolytic Capacitor")
@@
       (stroke (width 0.1) (type solid)) (fill none) (layer "F.Fab"))
     (pad "1" thru_hole rect (at 0 0 90) (size 2.8 2.8) (drill 1.4) (layers "*.Cu" "*.Mask")
-      (net 58 "Net-(D301-K)") (pinfunction "K") (pintype "passive"))
+      (net 58 "/converter/Vsnub") (pinfunction "K") (pintype "passive"))
     (pad "2" thru_hole oval (at 5.08 0 90) (size 2.8 2.8) (drill 1.4) (layers "*.Cu" "*.Mask")
       (net 29 "/V_SW") (pinfunction "A") (pintype "passive"))
@@
       (net 2 "GND") (pinfunction "2") (pintype "passive"))
   )
+  (footprint "Capacitor_THT:C_Radial_D10.0mm_H16.0mm_P5.00mm" (layer "F.Cu")
+    (at 174.7 114.475)
+    (descr "C, Radial series, Radial, pin pitch=5.00mm, diameter=10mm, height=16mm, Non-Polar Electrolytic Capacitor")
+    (tags "C Radial series Radial pin pitch 5.00mm diameter 10mm height 16mm Non-Polar Electrolytic Capacitor")
+    (property "Distributor" "Mouser")
+    (property "JLC P/N" "")
+    (property "Manufacturer" "KEMET")
+    (property "P/N" "80-A759MS186M2CAAE90")
+    (property "Sheetfile" "converter.kicad_sch")
+    (property "Sheetname" "converter")
+    (property "ki_description" "Unpolarized capacitor")
+    (property "ki_keywords" "cap capacitor")
+    (attr through_hole)
+    (fp_text reference "C305" (at 2.5 -6.25) (layer "F.SilkS")
+        (effects (font (size 1 1) (thickness 0.15)))
+    )
+    (fp_text value "18uF" (at 2.5 6.25) (layer "F.Fab")
+        (effects (font (size 1 1) (thickness 0.15)))
+    )
+    (fp_text user "${REFERENCE}" (at 2.5 0) (layer "F.Fab")
+        (effects (font (size 1 1) (thickness 0.15)))
+    )
+    (fp_circle (center 2.5 0) (end 7.62 0)
+      (stroke (width 0.12) (type solid)) (fill none) (layer "F.SilkS"))
+    (fp_circle (center 2.5 0) (end 7.75 0)
+      (stroke (width 0.05) (type solid)) (fill none) (layer "F.CrtYd"))
+    (fp_circle (center 2.5 0) (end 7.5 0)
+      (stroke (width 0.1) (type solid)) (fill none) (layer "F.Fab"))
+    (pad "1" thru_hole circle (at 0 0) (size 1.6 1.6) (drill 0.8) (layers "*.Cu" "*.Mask")
+      (net 4 "/V_BATT+") (pintype "passive"))
+    (pad "2" thru_hole circle (at 5 0) (size 1.6 1.6) (drill 0.8) (layers "*.Cu" "*.Mask")
+      (net 2 "GND") (pintype "passive"))
+    (model "${KICAD6_3DMODEL_DIR}/Capacitor_THT.3dshapes/C_Radial_D10.0mm_H16.0mm_P5.00mm.wrl"
+      (offset (xyz 0 0 0))
+      (scale (xyz 1 1 1))
+      (rotate (xyz 0 0 0))
+    )
+  )
   (footprint "mppt:EPC2307" (layer "F.Cu")
     (at 164.423697 98.39875)
@@
     )
   )
+  (footprint "Resistor_SMD:R_0805_2012Metric" (layer "F.Cu")
+    (at 172.775 90.1125 -90)
+    (descr "Resistor SMD 0805 (2012 Metric), square (rectangular) end terminal, IPC_7351 nominal, (Body size source: IPC-SM-782 page 72, https://www.pcb-3d.com/wordpress/wp-content/uploads/ipc-sm-782a_amendment_1_and_2.pdf), generated with kicad-footprint-generator")
+    (tags "resistor")
+    (property "Distributor" "Digikey")
+    (property "Manufacturer" "Kyocera AVX")
+    (property "P/N" "QB0805B40WYT")
+    (property "Sheetfile" "mppt.kicad_sch")
+    (property "Sheetname" "")
+    (property "ki_description" "Solder Jumper, 2-pole, closed/bridged")
+    (property "ki_keywords" "solder jumper SPST")
+    (attr smd)
+    (fp_text reference "TJ104" (at 0 -1.65 90) (layer "F.SilkS")
+        (effects (font (size 1 1) (thickness 0.15)))
+    )
+    (fp_text value "Thermal Jumper" (at 0 1.65 90) (layer "F.Fab")
+        (effects (font (size 1 1) (thickness 0.15)))
+    )
+    (fp_text user "${REFERENCE}" (at 0 0 90) (layer "F.Fab")
+        (effects (font (size 0.5 0.5) (thickness 0.08)))
+    )
+    (fp_line (start -0.227064 -0.735) (end 0.227064 -0.735)
+      (stroke (width 0.12) (type solid)) (layer "F.SilkS"))
+    (fp_line (start -0.227064 0.735) (end 0.227064 0.735)
+      (stroke (width 0.12) (type solid)) (layer "F.SilkS"))
+    (fp_line (start -1.68 -0.95) (end 1.68 -0.95)
+      (stroke (width 0.05) (type solid)) (layer "F.CrtYd"))
+    (fp_line (start -1.68 0.95) (end -1.68 -0.95)
+      (stroke (width 0.05) (type solid)) (layer "F.CrtYd"))
+    (fp_line (start 1.68 -0.95) (end 1.68 0.95)
+      (stroke (width 0.05) (type solid)) (layer "F.CrtYd"))
+    (fp_line (start 1.68 0.95) (end -1.68 0.95)
+      (stroke (width 0.05) (type solid)) (layer "F.CrtYd"))
+    (fp_line (start -1 -0.625) (end 1 -0.625)
+      (stroke (width 0.1) (type solid)) (layer "F.Fab"))
+    (fp_line (start -1 0.625) (end -1 -0.625)
+      (stroke (width 0.1) (type solid)) (layer "F.Fab"))
+    (fp_line (start 1 -0.625) (end 1 0.625)
+      (stroke (width 0.1) (type solid)) (layer "F.Fab"))
+    (fp_line (start 1 0.625) (end -1 0.625)
+      (stroke (width 0.1) (type solid)) (layer "F.Fab"))
+    (pad "1" smd roundrect (at -0.9125 0 270) (size 1.025 1.4) (layers "F.Cu" "F.Paste" "F.Mask") (roundrect_rratio 0.243902)
+      (net 1 "+12V") (pinfunction "A") (pintype "passive"))
+    (pad "2" smd roundrect (at 0.9125 0 270) (size 1.025 1.4) (layers "F.Cu" "F.Paste" "F.Mask") (roundrect_rratio 0.243902)
+      (net 4 "/V_BATT+") (pinfunction "B") (pintype "passive"))
+    (model "${KICAD6_3DMODEL_DIR}/Resistor_SMD.3dshapes/R_0805_2012Metric.wrl"
+      (offset (xyz 0 0 0))
+      (scale (xyz 1 1 1))
+      (rotate (xyz 0 0 0))
+    )
+  )
   (footprint "TestPoint:TestPoint_Keystone_5000-5004_Miniature" (layer "F.Cu")
     (at 98 111.7)
@@
     )
     (pad "1" thru_hole circle (at 0 -1.27 180) (size 1.5 1.5) (drill 1) (layers "*.Cu" "*.Mask")
-      (net 58 "Net-(D301-K)") (pinfunction "1") (pintype "passive"))
+      (net 58 "/converter/Vsnub") (pinfunction "1") (pintype "passive"))
     (pad "2" thru_hole circle (at 0 1.27 180) (size 2.6 2.6) (drill 2) (layers "*.Cu" "*.Mask")
       (net 2 "GND") (pinfunction "2") (pintype "passive"))
   )
   (footprint "TestPoint:TestPoint_Keystone_5000-5004_Miniature" (layer "F.Cu")
-    (at 182.08 111.68)
+    (at 186.4 110.225)
     (descr "Keystone Miniature THM Test Point 5000-5004, http://www.keyelco.com/product-pdf.cfm?p=1309")
     (tags "Through Hole Mount Test Points")
@@
       (stroke (width 0.1) (type solid)) (fill none) (layer "B.Fab"))
     (pad "1" thru_hole circle (at 0 0) (size 1.6 1.6) (drill 0.8) (layers "*.Cu" "*.Mask")
-      (net 58 "Net-(D301-K)") (pintype "passive"))
+      (net 58 "/converter/Vsnub") (pintype "passive"))
     (pad "2" thru_hole circle (at 5 0) (size 1.6 1.6) (drill 0.8) (layers "*.Cu" "*.Mask")
       (net 2 "GND") (pintype "passive"))
@@
       (net 29 "/V_SW") (pintype "passive"))
     (pad "2" thru_hole circle (at 5 0 270) (size 2.4 2.4) (drill 1.2) (layers "*.Cu" "*.Mask")
-      (net 58 "Net-(D301-K)") (pintype "passive"))
+      (net 58 "/converter/Vsnub") (pintype "passive"))
     (model "${KICAD6_3DMODEL_DIR}/Resistor_THT.3dshapes/R_Radial_Power_L11.0mm_W7.0mm_P5.00mm.wrl"
       (offset (xyz 0 0 0))
@@
   (segment (start 177.25 96.05) (end 177.25 102.65) (width 0.25) (layer "In1.Cu") (net 6))
   (segment (start 177.25 94.6) (end 177.25 96.05) (width 0.25) (layer "B.Cu") (net 6))
-  (segment (start 182.1 111.6) (end 182.1 107.6) (width 0.25) (layer "B.Cu") (net 6))
-  (segment (start 182.1 107.6) (end 184.5 105.2) (width 0.25) (layer "B.Cu") (net 6))
+  (segment (start 186.4 107.1) (end 186.4 110.225) (width 0.25) (layer "B.Cu") (net 6))
+  (segment (start 184.5 105.2) (end 186.4 107.1) (width 0.25) (layer "B.Cu") (net 6))
   (segment (start 161.005 95.31375) (end 160.265 94.57375) (width 0.25) (layer "F.Cu") (net 7))
   (segment (start 161.055 96.13375) (end 161.295 96.37375) (width 0.25) (layer "F.Cu") (net 7))
