File: hw/power_reg.kicad_sch (KiCad schematic)
At the start: 8 parts, among them J301 43650-0227

Commit message: savestate
Changed lines of the file:
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@@
     (stroke (width 0) (type default))
   )
-  (text_box "12V to 12V. Isolated."
+  (text_box "12V to 12V. Nonisolated."
     (at 120.65 58.42 0) (size 39.37 3.81)
     (stroke (width 0) (type default))
