File: hw/actuators.kicad_sch (KiCad schematic)
At the start: 10 parts, among them M1 5V, Q1 NMOS

Commit message: v0.3.0rc (v1.0.0rc) sch complete
Parts:
- added R20, R21: R_Small, symbol Device:R_Small
Connections:
- net FAN: now also R20.1, R21.1; no longer Q1.2 (G)
- net GND: now also R21.2
- new net: Q1.2 (G), R20.2
Other:
- note added: "Mounting points placed on FETs and gate driver as done on v0.1.0"
- note added: "Need to select slew resistor and pulldown, double check circuit"
- company: (none) -> LHR Solar
- title: (none) -> Sunscatter MPPT
Changed lines of the file:
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@@
 	(generator_version "8.0")
 	(paper "A4")
+	(title_block
+		(title "Sunscatter MPPT")
+		(date "2024-05-03")
+		(rev "v0.3.0rc")
+		(company "LHR Solar")
+		(comment 1 "Matthew Yu")
+		(comment 2 "Jacob Pustilnik")
+		(comment 3 "Gary Hallock")
+	)
+	(junction
+		(at 110.49 124.46)
+		(diameter 0)
+		(color 0 0 0 0)
+	)
 	(junction
 		(at 139.7 93.98)
@@
 	(wire
 		(pts
+			(xy 110.49 124.46) (xy 114.3 124.46)
+		)
+		(stroke
+			(width 0)
+			(type default)
+		)
+	)
+	(wire
+		(pts
 			(xy 129.54 119.38) (xy 129.54 118.11)
 		)
@@
 	(wire
 		(pts
+			(xy 119.38 124.46) (xy 121.92 124.46)
+		)
+		(stroke
+			(width 0)
+			(type default)
+		)
+	)
+	(wire
+		(pts
 			(xy 139.7 118.11) (xy 129.54 118.11)
 		)
@@
 	(wire
 		(pts
+			(xy 107.95 124.46) (xy 110.49 124.46)
+		)
+		(stroke
+			(width 0)
+			(type default)
+		)
+	)
+	(wire
+		(pts
 			(xy 139.7 109.22) (xy 139.7 118.11)
 		)
@@
 		(pts
 			(xy 139.7 93.98) (xy 129.54 93.98)
+		)
+		(stroke
+			(width 0)
+			(type default)
+		)
+	)
+	(wire
+		(pts
+			(xy 110.49 129.54) (xy 129.54 129.54)
 		)
 		(stroke
@@
 		)
 	)
-	(hierarchical_label "FAN"
-		(shape input)
-		(at 121.92 124.46 180)
-		(fields_autoplaced yes)
+	(text "Mounting points placed on FETs \nand gate driver as done on v0.1.0"
+		(exclude_from_sim no)
+		(at 109.728 105.41 0)
 		(effects
 			(font
 				(size 1.27 1.27)
 			)
+		)
+	)
+	(text "Need to select slew resistor and \npulldown, double check circuit"
+		(exclude_from_sim no)
+		(at 95.504 119.888 0)
+		(effects
+			(font
+				(size 1.27 1.27)
+			)
+		)
+	)
+	(hierarchical_label "FAN"
+		(shape input)
+		(at 107.95 124.46 180)
+		(fields_autoplaced yes)
+		(effects
+			(font
+				(size 1.27 1.27)
+			)
 			(justify right)
+		)
+	)
+	(symbol
+		(lib_id "Device:R_Small")
+		(at 116.84 124.46 90)
+		(unit 1)
+		(exclude_from_sim no)
+		(in_bom yes)
+		(on_board yes)
+		(dnp no)
+		(fields_autoplaced yes)
+		(property "Reference" "R20"
+			(at 116.84 119.38 90)
+			(effects
+				(font
+					(size 1.27 1.27)
+				)
+			)
+		)
+		(property "Value" "R_Small"
+			(at 116.84 121.92 90)
+			(effects
+				(font
+					(size 1.27 1.27)
+				)
+			)
+		)
+		(property "Footprint" ""
+			(at 116.84 124.46 0)
+			(effects
+				(font
+					(size 1.27 1.27)
+				)
+				(hide yes)
+			)
+		)
+		(property "Datasheet" "~"
+			(at 116.84 124.46 0)
+			(effects
+				(font
+					(size 1.27 1.27)
+				)
+				(hide yes)
+			)
+		)
+		(property "Description" "Resistor, small symbol"
+			(at 116.84 124.46 0)
+			(effects
+				(font
+					(size 1.27 1.27)
+				)
+				(hide yes)
+			)
+		)
+		(pin "2"
+		)
+		(pin "1"
+		)
+		(instances
+			(project "mppt"
+				(path "/06fd3a42-664d-41bc-bf0f-b5ee0ddcc902/e1f5a50e-a1f9-4d2e-b822-1c90ec1f58b5"
+					(reference "R20")
+					(unit 1)
+				)
+			)
 		)
 	)
@@
 					(unit 1)
 				)
+			)
+		)
+	)
+	(symbol
+		(lib_id "Device:R_Small")
+		(at 110.49 127 0)
+		(unit 1)
+		(exclude_from_sim no)
+		(in_bom yes)
+		(on_board yes)
+		(dnp no)
+		(fields_autoplaced yes)
+		(property "Reference" "R21"
+			(at 113.03 125.7299 0)
+			(effects
+				(font
+					(size 1.27 1.27)
+				)
+				(justify left)
+			)
+		)
+		(property "Value" "R_Small"
+			(at 113.03 128.2699 0)
+			(effects
+				(font
+					(size 1.27 1.27)
+				)
+				(justify left)
+			)
+		)
+		(property "Footprint" ""
+			(at 110.49 127 0)
+			(effects
+				(font
+					(size 1.27 1.27)
+				)
+				(hide yes)
+			)
+		)
+		(property "Datasheet" "~"
+			(at 110.49 127 0)
+			(effects
+				(font
+					(size 1.27 1.27)
+				)
+				(hide yes)
+			)
+		)
+		(property "Description" "Resistor, small symbol"
+			(at 110.49 127 0)
+			(effects
+				(font
+					(size 1.27 1.27)
+				)
+				(hide yes)
+			)
+		)
+		(pin "2"
+		)
+		(pin "1"
+		)
+		(instances
+			(project "mppt"
+				(path "/06fd3a42-664d-41bc-bf0f-b5ee0ddcc902/e1f5a50e-a1f9-4d2e-b822-1c90ec1f58b5"
+					(reference "R21")
+					(unit 1)
+				)
