File: hw/gate_driver.kicad_sch (KiCad schematic)
At the start: 14 parts, among them U501 LMG1210RVRT

Commit message: fixes for v0.1.1rc
Other:
- company: (none) -> UT LHR Solar
- title: MPPT -> Sunscatter MPPT
Changed lines of the file:
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@@
   (paper "A4")
   (title_block
-    (title "MPPT")
-    (date "2023-01-30")
-    (rev "v0.0.0")
-    (comment 1 "Nishant Gupta")
+    (title "Sunscatter MPPT")
+    (date "2023-03-26")
+    (rev "v0.1.1")
+    (company "UT LHR Solar")
+    (comment 1 "Matthew Yu")
     (comment 2 "Jacob Pustilnik")
   )

Commit message: updated instructions for v0.2.0 - v0.5.0 development candidates.
Parts:
- C201: Cost (none) -> 0.0068; JLC P/N C307331 -> (none)
- C501, C505: Cost (none) -> 0.0234; JLC P/N C96446 -> (none)
- C503: Cost (none) -> 0.0039; JLC P/N C52923 -> (none)
- D501: Cost (none) -> 0.42
- R501, R502: Cost (none) -> 0.0005; JLC P/N C25765 -> (none)
- R503, R504: Cost (none) -> 0.0009; JLC P/N C423254 -> (none)
- U501: Cost (none) -> 4.077
Changed lines of the file:
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@@
   (title_block
     (title "Sunscatter MPPT")
-    (date "2023-03-26")
-    (rev "v0.1.1")
+    (date "2023-04-18")
+    (rev "v0.1.1rc")
     (company "UT LHR Solar")
     (comment 1 "Matthew Yu")
@@
       (effects (font (size 1.27 1.27)) hide)
     )
-    (property "JLC P/N" "C423254" (at 181.61 99.06 0)
-      (effects (font (size 1.27 1.27)) hide)
-    )
     (property "Manufacturer" "Uniroyal Elec" (at 181.61 99.06 0)
       (effects (font (size 1.27 1.27)) hide)
@@
       (effects (font (size 1.27 1.27)) hide)
     )
+    (property "Cost" "0.0009" (at 181.61 99.06 0)
+      (effects (font (size 1.27 1.27)) hide)
+    )
     (pin "1")
     (pin "2")
@@
       (effects (font (size 1.27 1.27)) hide)
     )
+    (property "Cost" "" (at 116.84 124.46 0)
+      (effects (font (size 1.27 1.27)) hide)
+    )
     (pin "1")
     (pin "2")
@@
       (effects (font (size 1.27 1.27)) hide)
     )
-    (property "JLC P/N" "C96446" (at 205.74 81.28 0)
-      (effects (font (size 1.27 1.27)) hide)
-    )
     (property "Manufacturer" "Samsung Electro-Mechanics" (at 205.74 81.28 0)
       (effects (font (size 1.27 1.27)) hide)
@@
     )
     (property "LCSC Part #" "C96446" (at 205.74 81.28 0)
+      (effects (font (size 1.27 1.27)) hide)
+    )
+    (property "Cost" "0.0234" (at 205.74 81.28 0)
       (effects (font (size 1.27 1.27)) hide)
     )
@@
       (effects (font (size 1.27 1.27)) hide)
     )
-    (property "JLC P/N" "C307331" (at 194.31 81.28 0)
-      (effects (font (size 1.27 1.27)) hide)
-    )
     (property "Manufacturer" "Samsung Electro-Mechanics" (at 194.31 81.28 0)
       (effects (font (size 1.27 1.27)) hide)
@@
     )
     (property "LCSC Part #" "C307331" (at 194.31 81.28 0)
+      (effects (font (size 1.27 1.27)) hide)
+    )
+    (property "Cost" "0.0068" (at 194.31 81.28 0)
       (effects (font (size 1.27 1.27)) hide)
     )
@@
       (effects (font (size 1.27 1.27)) hide)
     )
-    (property "JLC P/N" "C423254" (at 181.61 93.98 0)
-      (effects (font (size 1.27 1.27)) hide)
-    )
     (property "Manufacturer" "Uniroyal Elec" (at 181.61 93.98 0)
       (effects (font (size 1.27 1.27)) hide)
@@
     )
     (property "LCSC Part #" "C423254" (at 181.61 93.98 0)
+      (effects (font (size 1.27 1.27)) hide)
+    )
+    (property "Cost" "0.0009" (at 181.61 93.98 0)
       (effects (font (size 1.27 1.27)) hide)
     )
@@
       (effects (font (size 1.27 1.27)) hide)
     )
-    (property "JLC P/N" "" (at 181.61 86.36 0)
-      (effects (font (size 1.27 1.27)) hide)
-    )
     (property "Manufacturer" "STMicroelectronics" (at 181.61 86.36 0)
       (effects (font (size 1.27 1.27)) hide)
@@
     )
     (property "LCSC Part #" "" (at 181.61 86.36 0)
+      (effects (font (size 1.27 1.27)) hide)
+    )
+    (property "Cost" "0.42" (at 181.61 86.36 0)
       (effects (font (size 1.27 1.27)) hide)
     )
@@
       (effects (font (size 1.27 1.27)) hide)
     )
-    (property "JLC P/N" "C52923" (at 128.27 104.14 0)
-      (effects (font (size 1.27 1.27)) hide)
-    )
     (property "Manufacturer" "Samsung Electro-Mechanics" (at 128.27 104.14 0)
       (effects (font (size 1.27 1.27)) hide)
@@
     )
     (property "LCSC Part #" "C52923" (at 128.27 104.14 0)
+      (effects (font (size 1.27 1.27)) hide)
+    )
+    (property "Cost" "0.0039" (at 128.27 104.14 0)
       (effects (font (size 1.27 1.27)) hide)
     )
@@
       (effects (font (size 1.27 1.27)) hide)
     )
-    (property "JLC P/N" "C96446" (at 110.49 81.28 0)
-      (effects (font (size 1.27 1.27)) hide)
-    )
     (property "Manufacturer" "Samsung Electro-Mechanics" (at 110.49 81.28 0)
       (effects (font (size 1.27 1.27)) hide)
@@
     )
     (property "LCSC Part #" "C96446" (at 110.49 81.28 0)
+      (effects (font (size 1.27 1.27)) hide)
+    )
+    (property "Cost" "0.0234" (at 110.49 81.28 0)
       (effects (font (size 1.27 1.27)) hide)
     )
@@
     )
     (property "LCSC Part #" "" (at 158.75 124.46 0)
+      (effects (font (size 1.27 1.27)) hide)
+    )
+    (property "Cost" "" (at 158.75 124.46 0)
       (effects (font (size 1.27 1.27)) hide)
     )
@@
       (effects (font (size 1.27 1.27)) hide)
     )
-    (property "JLC P/N" "C25765" (at 108.585 96.52 0)
-      (effects (font (size 1.27 1.27)) hide)
-    )
     (property "Manufacturer" "Uniroyal Elec" (at 108.585 96.52 0)
       (effects (font (size 1.27 1.27)) hide)
@@
     )
     (property "LCSC Part #" "C25765" (at 108.585 96.52 0)
+      (effects (font (size 1.27 1.27)) hide)
+    )
+    (property "Cost" "0.0005" (at 108.585 96.52 0)
       (effects (font (size 1.27 1.27)) hide)
     )
@@
       (effects (font (size 1.27 1.27)) hide)
     )
-    (property "JLC P/N" "" (at 156.21 96.52 0)
-      (effects (font (size 1.27 1.27)) hide)
-    )
     (property "Manufacturer" "Texas Instruments" (at 156.21 96.52 0)
       (effects (font (size 1.27 1.27)) hide)
@@
     )
     (property "LCSC Part #" "" (at 156.21 96.52 0)
+      (effects (font (size 1.27 1.27)) hide)
+    )
+    (property "Cost" "4.077" (at 156.21 96.52 0)
       (effects (font (size 1.27 1.27)) hide)
     )
@@
       (effects (font (size 1.27 1.27)) hide)
     )
+    (property "Cost" "" (at 138.43 124.46 0)
+      (effects (font (size 1.27 1.27)) hide)
+    )
     (pin "1")
     (pin "2")
@@
       (effects (font (size 1.27 1.27)) hide)
     )
-    (property "JLC P/N" "C25765" (at 100.33 93.98 0)
-      (effects (font (size 1.27 1.27)) hide)
-    )
     (property "Manufacturer" "Uniroyal Elec" (at 100.33 93.98 0)
       (effects (font (size 1.27 1.27)) hide)
@@
     )
     (property "LCSC Part #" "C25765" (at 100.33 93.98 0)
+      (effects (font (size 1.27 1.27)) hide)
+    )
+    (property "Cost" "0.0005" (at 100.33 93.98 0)
       (effects (font (size 1.27 1.27)) hide)
     )
@@
       (effects (font (size 1.27 1.27)) hide)
     )
-    (property "JLC P/N" "C307331" (at 120.65 81.28 0)
-      (effects (font (size 1.27 1.27)) hide)
-    )
     (property "Manufacturer" "Samsung Electro-Mechanics" (at 120.65 81.28 0)
       (effects (font (size 1.27 1.27)) hide)
@@
       (effects (font (size 1.27 1.27)) hide)
     )
+    (property "Cost" "0.0068" (at 120.65 81.28 0)
+      (effects (font (size 1.27 1.27)) hide)
+    )

Commit message: hw changes
Parts:
- D501: footprint mppt:SODFL5226X110N -> footprints:SODFL5226X110N
- TP501, TP502, TP503: footprint mppt:SignalTP -> footprints:SignalTP
- U501: footprint mppt:IC_LMG1210RVRT -> footprints:IC_LMG1210RVRT
Other:
- moved on the sheet: R502
Changed lines of the file:
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@@
     (stroke (width 0) (type default))
   )
-  (wire (pts (xy 108.585 93.98) (xy 138.43 93.98))
+  (wire (pts (xy 109.22 93.98) (xy 138.43 93.98))
     (stroke (width 0) (type default))
   )
@@
       (effects (font (size 1 1)) (justify left))
     )
-    (property "Footprint" "mppt:SignalTP" (at 116.84 124.46 0)
+    (property "Footprint" "footprints:SignalTP" (at 116.84 124.46 0)
       (effects (font (size 1.27 1.27)) hide)
     )
@@
       (effects (font (size 1 1)) (justify left))
     )
-    (property "Footprint" "mppt:SODFL5226X110N" (at 181.61 86.36 0)
+    (property "Footprint" "footprints:SODFL5226X110N" (at 181.61 86.36 0)
       (effects (font (size 1.27 1.27)) hide)
     )
@@
       (effects (font (size 1 1)) (justify left))
     )
-    (property "Footprint" "mppt:SignalTP" (at 158.75 124.46 0)
+    (property "Footprint" "footprints:SignalTP" (at 158.75 124.46 0)
       (effects (font (size 1.27 1.27)) hide)
     )
@@
     )
   )
-  (symbol (lib_id "Device:R_Small") (at 108.585 96.52 0) (unit 1)
+  (symbol (lib_id "Device:R_Small") (at 109.22 96.52 0) (unit 1)
     (in_bom yes) (on_board yes) (dnp no)
-    (property "Reference" "R502" (at 111.125 95.885 0)
-      (effects (font (size 1 1)) (justify left))
-    )
-    (property "Value" "20k" (at 111.125 98.425 0)
-      (effects (font (size 1 1)) (justify left))
-    )
-    (property "Footprint" "Resistor_SMD:R_0402_1005Metric" (at 108.585 96.52 0)
-      (effects (font (size 1.27 1.27)) hide)
-    )
-    (property "Datasheet" "https://datasheet.lcsc.com/lcsc/2206010100_UNI-ROYAL-Uniroyal-Elec-0402WGF2002TCE_C25765.pdf" (at 108.585 96.52 0)
-      (effects (font (size 1.27 1.27)) hide)
-    )
-    (property "Distributor" "JLCPCB" (at 108.585 96.52 0)
-      (effects (font (size 1.27 1.27)) hide)
-    )
-    (property "Manufacturer" "Uniroyal Elec" (at 108.585 96.52 0)
-      (effects (font (size 1.27 1.27)) hide)
-    )
-    (property "P/N" "0402WGF2002TCE" (at 108.585 96.52 0)
-      (effects (font (size 1.27 1.27)) hide)
-    )
-    (property "LCSC Part #" "C25765" (at 108.585 96.52 0)
-      (effects (font (size 1.27 1.27)) hide)
-    )
-    (property "Cost" "0.0005" (at 108.585 96.52 0)
+    (property "Reference" "R502" (at 111.76 95.885 0)
+      (effects (font (size 1 1)) (justify left))
+    )
+    (property "Value" "20k" (at 111.76 98.425 0)
+      (effects (font (size 1 1)) (justify left))
+    )
+    (property "Footprint" "Resistor_SMD:R_0402_1005Metric" (at 109.22 96.52 0)
+      (effects (font (size 1.27 1.27)) hide)
+    )
+    (property "Datasheet" "https://datasheet.lcsc.com/lcsc/2206010100_UNI-ROYAL-Uniroyal-Elec-0402WGF2002TCE_C25765.pdf" (at 109.22 96.52 0)
+      (effects (font (size 1.27 1.27)) hide)
+    )
+    (property "Distributor" "JLCPCB" (at 109.22 96.52 0)
+      (effects (font (size 1.27 1.27)) hide)
+    )
+    (property "Manufacturer" "Uniroyal Elec" (at 109.22 96.52 0)
+      (effects (font (size 1.27 1.27)) hide)
+    )
+    (property "P/N" "0402WGF2002TCE" (at 109.22 96.52 0)
+      (effects (font (size 1.27 1.27)) hide)
+    )
+    (property "LCSC Part #" "C25765" (at 109.22 96.52 0)
+      (effects (font (size 1.27 1.27)) hide)
+    )
+    (property "Cost" "0.0005" (at 109.22 96.52 0)
       (effects (font (size 1.27 1.27)) hide)
     )
@@
       (effects (font (size 1 1)))
     )
-    (property "Footprint" "mppt:IC_LMG1210RVRT" (at 156.21 96.52 0)
+    (property "Footprint" "footprints:IC_LMG1210RVRT" (at 156.21 96.52 0)
       (effects (font (size 1.27 1.27)) (justify bottom) hide)
     )
@@
       (effects (font (size 1 1)) (justify left))
     )
-    (property "Footprint" "mppt:SignalTP" (at 138.43 124.46 0)
+    (property "Footprint" "footprints:SignalTP" (at 138.43 124.46 0)
       (effects (font (size 1.27 1.27)) hide)
     )
@@
     )
   )
-  (symbol (lib_id "power:GND") (at 108.585 99.06 0) (unit 1)
+  (symbol (lib_id "power:GND") (at 109.22 99.06 0) (unit 1)
     (in_bom yes) (on_board yes) (dnp no)
-    (property "Reference" "#PWR0505" (at 108.585 105.41 0)
+    (property "Reference" "#PWR0505" (at 109.22 105.41 0)
       (effects (font (size 1 1)) hide)
     )
-    (property "Value" "GND" (at 108.585 102.87 0)
-      (effects (font (size 1 1)))
-    )
-    (property "Footprint" "" (at 108.585 99.06 0)
-      (effects (font (size 1.27 1.27)) hide)
-    )
-    (property "Datasheet" "" (at 108.585 99.06 0)
-      (effects (font (size 1.27 1.27)) hide)
-    )
+    (property "Value" "GND" (at 109.22 102.87 0)
+      (effects (font (size 1 1)))
+    )
+    (property "Footprint" "" (at 109.22 99.06 0)
+      (effects (font (size 1.27 1.27)) hide)
+    )
+    (property "Datasheet" "" (at 109.22 99.06 0)
+      (effects (font (size 1.27 1.27)) hide)
+    )

Commit message: v0.2.0
Parts:
- removed C201 (x2): 100nF, Capacitor_SMD:C_0402_1005Metric, symbol Device:C_Small
- removed TP501, TP502, TP503: TestPoint_2Pole, footprints:SignalTP, symbol Connector:TestPoint_2Pole
- removed U501: LMG1210RVRT, footprints:IC_LMG1210RVRT, symbol LMG1210RVRT:LMG1210RVRT
- added C201 (x2): 100nF, Capacitor_SMD:C_0402_1005Metric, symbol Device:C_Small
- added IC501: LMG1210RVRT, footprints:ti_LMG1210RVRT, symbol ti_LMG1210RVRT:LMG1210RVRT
- added TP501: SW1_TP, TestPoint:TestPoint_Keystone_5005-5009_Compact, symbol Connector:TestPoint
- added TP502: GND_TP, TestPoint:TestPoint_Keystone_5005-5009_Compact, symbol Connector:TestPoint
- added TP503: SW2_TP, TestPoint:TestPoint_Keystone_5005-5009_Compact, symbol Connector:TestPoint
- added TP504: PWMEN_TP, TestPoint:TestPoint_Pad_1.0x1.0mm, symbol Connector:TestPoint
- added TP505: PWM_TP, TestPoint:TestPoint_Pad_1.0x1.0mm, symbol Connector:TestPoint
- C503: value 1uF -> 10uF; footprint Capacitor_SMD:C_0402_1005Metric -> Capacitor_SMD:C_0603_1608Metric; Cost 0.0039 -> 0.0234; LCSC Part # C52923 -> C96446; P/N CL05A105KA5NQNC -> CL10A106MA8NRNC
- C505: value 10uF -> 1uF; footprint Capacitor_SMD:C_0603_1608Metric -> Capacitor_SMD:C_0402_1005Metric; Cost 0.0234 -> 0.0039; LCSC Part # C96446 -> C52923; P/N CL10A106MA8NRNC -> CL05A105KA5NQNC
- D501: value 0.62V Schottky -> 0.62V; footprint footprints:SODFL5226X110N -> footprints:stm_STPS1170AF
- R502: value 20k -> 1.8; Cost 0.0005 -> 0.0009; LCSC Part # C25765 -> C423254; P/N 0402WGF2002TCE -> 0402WGF118KTCE
- R503: value 1.8 -> 20k; Cost 0.0009 -> 0.0005; LCSC Part # C423254 -> C25765; P/N 0402WGF118KTCE -> 0402WGF2002TCE
Connections:
- net DHL is gone; now on net SW1_OUT: R502.1
- net HO is gone; now on net SW2_OUT: R504.1
- net LO is gone; now on net GND: R503.1
- net +12V: now also C503.1, C201.1, IC501.2 (VIN); no longer C501.1
- net +5V: now also C501.1, C201.1, IC501.4 (VDD); no longer C505.1
- net GND: now also C503.2, C201.2, C201.2, IC501.20 (VSS_3), IC501.3 (VSS_1), IC501.7 (VSS_2), TP502.1; no longer C505.2, R502.2
- net PWM: now also IC501.19 (PWM/LI), TP505.1
- net PWM_EN: now also IC501.18 (EN/HI), TP504.1
- net SW1_OUT: now also TP501.1; no longer R503.2
- net SW2_OUT: now also TP503.1; no longer R504.2
- net V_SW: now also C505.2, IC501.13 (HS_2), IC501.16 (HS_3), IC501.21 (HS_4), IC501.9 (HS_1); no longer C503.1
- net BST: no longer names the net of D501.2 (A)
- net BST: now also IC501.17 (BST)
- net DLH: no longer names the net of R501.1
- net DLH: now also IC501.5 (DHL)
- net HB: no longer names the net of D501.1 (K)
- net HB: now also C505.1, IC501.12 (HB); no longer C503.2
- new net: IC501.8 (LO), R502.2
- new net: IC501.1 (NC_1), IC501.11 (NC_2), IC501.14 (NC1), IC501.15 (NC_3)
- new net: IC501.10 (HO), R504.2
- new net: IC501.6 (DLH), R503.2
- no-connect marks 1 -> 0
Other:
- note added: "Gate Driver"
- company: UT LHR Solar -> LHR Solar

Commit message: bugfix for wrong adc pin for batt current measurements
Parts:
- C201: Cost 0.0068 -> 0.0063; LCSC Part # C307331 -> CL05B104KB54PNC; Notes (none) -> Rated for 50V.
Changed lines of the file:
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@@
       (effects (font (size 1 1)) hide)
     )
-    (property "Datasheet" "~" (at 142.24 123.19 0)
+    (property "Datasheet" "" (at 142.24 123.19 0)
       (effects (font (size 1 1)) hide)
     )
@@
       (effects (font (size 1 1)) hide)
     )
-    (property "Datasheet" "~" (at 154.94 123.19 0)
+    (property "Datasheet" "" (at 154.94 123.19 0)
       (effects (font (size 1 1)) hide)
     )
@@
       (effects (font (size 1 1)) hide)
     )
-    (property "Datasheet" "~" (at 129.54 123.19 0)
+    (property "Datasheet" "" (at 129.54 123.19 0)
       (effects (font (size 1 1)) hide)
     )
@@
       (effects (font (size 1 1)) hide)
     )
-    (property "Datasheet" "https://datasheet.lcsc.com/lcsc/1810191222_Samsung-Electro-Mechanics-CL05B104KB54PNC_C307331.pdf" (at 106.68 91.44 0)
+    (property "Datasheet" "https://datasheet.lcsc.com/lcsc/2304140030_Samsung-Electro-Mechanics-CL05B104KB54PNC_C307331.pdf" (at 106.68 91.44 0)
       (effects (font (size 1 1)) hide)
     )
@@
       (effects (font (size 1 1)) hide)
     )
-    (property "LCSC Part #" "C307331" (at 106.68 91.44 0)
-      (effects (font (size 1 1)) hide)
-    )
-    (property "Cost" "0.0068" (at 106.68 91.44 0)
-      (effects (font (size 1 1)) hide)
+    (property "LCSC Part #" "CL05B104KB54PNC" (at 106.68 91.44 0)
+      (effects (font (size 1 1)) hide)
+    )
+    (property "Cost" "0.0063" (at 106.68 91.44 0)
+      (effects (font (size 1 1)) hide)
+    )
+    (property "Notes" "Rated for 50V." (at 106.68 91.44 0)
+      (effects (font (size 1.27 1.27)) hide)
     )
     (pin "1")
@@
       (effects (font (size 1 1)) hide)
     )
-    (property "Datasheet" "~" (at 118.11 135.89 0)
+    (property "Datasheet" "" (at 118.11 135.89 0)
       (effects (font (size 1 1)) hide)
     )
@@
       (effects (font (size 1 1)) hide)
     )
-    (property "Datasheet" "https://datasheet.lcsc.com/lcsc/1810191222_Samsung-Electro-Mechanics-CL05B104KB54PNC_C307331.pdf" (at 124.46 91.44 0)
+    (property "Datasheet" "https://datasheet.lcsc.com/lcsc/2304140030_Samsung-Electro-Mechanics-CL05B104KB54PNC_C307331.pdf" (at 124.46 91.44 0)
       (effects (font (size 1 1)) hide)
     )
@@
       (effects (font (size 1 1)) hide)
     )
-    (property "LCSC Part #" "C307331" (at 124.46 91.44 0)
-      (effects (font (size 1 1)) hide)
-    )
-    (property "Cost" "0.0068" (at 124.46 91.44 0)
-      (effects (font (size 1 1)) hide)
+    (property "LCSC Part #" "CL05B104KB54PNC" (at 124.46 91.44 0)
+      (effects (font (size 1 1)) hide)
+    )
+    (property "Cost" "0.0063" (at 124.46 91.44 0)
+      (effects (font (size 1 1)) hide)
+    )
+    (property "Notes" "Rated for 50V." (at 124.46 91.44 0)
+      (effects (font (size 1.27 1.27)) hide)
     )
     (pin "1")
@@
       (effects (font (size 1 1)) hide)
     )
-    (property "Datasheet" "~" (at 118.11 123.19 0)
-      (effects (font (size 1 1)) hide)
-    )
+    (property "Datasheet" "" (at 118.11 123.19 0)
+      (effects (font (size 1 1)) hide)
+    )

Commit message: init sch changes
Parts:
- removed C201: 100nF, Capacitor_SMD:C_0402_1005Metric, symbol Device:C_Small
- removed C503: 10uF, Capacitor_SMD:C_0603_1608Metric, symbol Device:C_Small
- removed TP502: GND_TP, TestPoint:TestPoint_Keystone_5005-5009_Compact, symbol Connector:TestPoint
- added TP19: GND, TestPoint:TestPoint_Pad_1.0x1.0mm, symbol Connector:TestPoint
- added TP8: 5V, TestPoint:TestPoint_Pad_1.0x1.0mm, symbol Connector:TestPoint
- renumbered C201 to C502
Connections:
- net +12V is gone; now on net +5V: IC501.2 (VIN)
- net +5V: now also TP8.1
- net GND: now also TP19.1
- net PWM renamed PWM/LI
- net PWM_EN renamed EN/HI
- net SW1_OUT renamed SWLO
- net SW2_OUT renamed SWHO
- net V_SW renamed V_{SW}
Other:
- moved on the sheet: C501, C502, TP501, TP503, TP504, TP505
