File: hw/power_regulation.kicad_sch (KiCad schematic)
At the start: 16 parts, among them IC1 LM74700QDBVRQ1, J1 43650-0227, Q2 NMOS, U2 AP63205WU, U4 LM1085-3.3

Commit message: v0.3.0rc (v1.0.0rc) sch complete
Parts:
- removed C11: 10uF, symbol Device:C_Small
- removed C12, C19: 100nF, symbol Device:C_Small
- removed C13, C14: 22uF, symbol Device:C_Small
- removed C18: 10uF, symbol Device:C_Polarized_Small
- removed D1: 12V, footprints:littelfuse_SZSMF4L12CAT3G, symbol littelfuse_SZSMF4L12CAT3G:SZSMF4L12CAT3G
- removed IC1: LM74700QDBVRQ1, SOT95P280X145-6N, symbol ti_LM74700QDBVRQ1:LM74700QDBVRQ1
- removed J1: 43650-0227, footprints:molex_microfit_43650_0227, symbol molex_microfit_43650_0227:43650-0227
- removed L1: 4.8uH, symbol Device:L_Small
- removed Q2: NMOS, symbol Simulation_SPICE:NMOS
- removed TP1, TP2, TP3: TestPoint, symbol Connector:TestPoint
- removed U2: AP63205WU, Package_TO_SOT_SMD:TSOT-23-6, symbol Regulator_Switching:AP63205WU
- removed U4: LM1085-3.3, symbol Regulator_Linear:LM1085-3.3
- added C701, C702, C707: 100n, Resistor_SMD:R_0402_1005Metric, symbol Device:C_Small
- added C703, C705: 10u, Resistor_SMD:R_0805_2012Metric, symbol Device:C_Small
- added C704, C706, C708, C712, C713: 1u, Resistor_SMD:R_0402_1005Metric, symbol Device:C_Small
- added C709, C710, C711: 22u, Resistor_SMD:R_0805_2012Metric, symbol Device:C_Small
- added C714: 4.7u, Resistor_SMD:R_0402_1005Metric, symbol Device:C_Small
- added D701: 15, Diode_SMD:D_SMA, symbol Diode:SMAJ15CA
- added D702, D703, D704, D705: GRN, LED_SMD:LED_0402_1005Metric, symbol Device:LED_Small
- added J701, J702: PWR Header, footprints:molex_microfit_43650_0227, symbol molex_microfit_43650_0227:43650-0227
- added JP701, JP702, JP703: Jumper_2_Bridged, Connector_PinHeader_2.54mm:PinHeader_1x02_P2.54mm_Vertical, symbol Jumper:Jumper_2_Bridged
- added L701: 4.7u, Inductor_SMD:L_TDK_VLS6045EX_VLS6045AF, symbol Device:L_Small
- added L702: 10u, Inductor_SMD:L_TDK_VLS6045EX_VLS6045AF, symbol Device:L_Small
- added Q701: Q_NMOS_GDS, Package_TO_SOT_SMD:SOT-223-3_TabPin2, symbol Device:Q_NMOS_GDS
- added R701: 3.3k, Resistor_SMD:R_0402_1005Metric, symbol Device:R_Small
- added R702, R705: 330, Resistor_SMD:R_0402_1005Metric, symbol Device:R_Small
- added R703: 0, Resistor_SMD:R_0402_1005Metric, symbol Device:R_Small
- added R704: 1k, Resistor_SMD:R_0402_1005Metric, symbol Device:R_Small
- added TP701: 12V, TestPoint:TestPoint_Keystone_5000-5004_Miniature, symbol Connector:TestPoint
- added TP702: 5V0, TestPoint:TestPoint_Keystone_5000-5004_Miniature, symbol Connector:TestPoint
- added TP703: 3V3, TestPoint:TestPoint_Keystone_5000-5004_Miniature, symbol Connector:TestPoint
- added TP704: 3V3P, TestPoint:TestPoint_Keystone_5000-5004_Miniature, symbol Connector:TestPoint
- added TP705: GND, TestPoint:TestPoint_Keystone_5000-5004_Miniature, symbol Connector:TestPoint
- added TP706: 5VP, TestPoint:TestPoint_Keystone_5000-5004_Miniature, symbol Connector:TestPoint
- added TP707: GNDPWR, TestPoint:TestPoint_Keystone_5000-5004_Miniature, symbol Connector:TestPoint
- added U701: LM74700-Q1, Package_TO_SOT_SMD:SOT-23-6, symbol Power_Management:LM74700
- added U702, U706: TLV75733, Package_TO_SOT_SMD:SOT-23-5, symbol Regulator_Linear:TLV75733PDBV
- added U703: AP63205WU, Package_TO_SOT_SMD:TSOT-23-6, symbol Regulator_Switching:AP63205WU
- added U704: TPS22917, Package_TO_SOT_SMD:SOT-23-6, symbol Power_Management:TPS22917DBV
- added U705: CRE1S0505, footprints:murata_CRE1S0505_MEC, symbol murata_CRE1S0505:CRE1S0505MEC-R
Connections:
- net +12V: now also C703.1, C705.1, Q701.2 (D), R701.1, TP701.1, U701.4 (CATHODE), U703.2 (EN), U703.3 (IN)
- net +3V3: now also C713.1, R705.1, TP703.1, U706.5 (OUT)
- net +5V: now also C704.1, C708.1, C712.1, JP701.2 (B), JP702.2 (B), JP703.2 (B), R704.1, TP702.1, U702.1 (IN), U704.1 (VIN), U706.1 (IN), U706.3 (EN)
- net GND: now also C701.2, C703.2, C704.2, C705.2, C706.2, C708.2, C709.2, C710.2, C711.2, C712.2, C713.2, D701.1 (A1), D702.1 (K), D703.1 (K), D704.1 (K), D705.1 (K), J701.2, J702.2, TP705.1, U701.2 (GND), U702.2 (GND), U703.4 (GND), U704.2 (GND), U705.1 (-VIN), U706.2 (GND)
- new net: D702.2 (A), R701.2
- new net: C701.1, C702.1, D701.2 (A2), J701.1, Q701.3 (S), U701.1 (VCAP), U701.6 (ANODE)
- new net: C702.2, U701.3 (EN)
- new net: Q701.1 (G), U701.5 (GATE)
- new net: C709.1, C710.1, JP701.1 (A), L701.2, U703.1 (FB)
- new net: C711.1, R703.1, U704.6 (VOUT), U705.3 (+VIN)
- new net: R703.2, U704.5 (QOD)
- new net: C707.1, U703.6 (BST)
- new net: C707.2, L701.1, U703.5 (SW)
- new net: D704.2 (A), R704.2
- new net: D705.2 (A), R705.2
- new net: D703.2 (A), R702.2
- new net: L702.1, U705.8 (+VOUT)
- new net: J702.1, JP703.1 (A)
- new net +3.3VP: C706.1, R702.1, TP704.1, U702.5 (OUT)
- new net +5VP: C714.1, L702.2, TP706.1
- new net GNDPWR: C714.2, TP707.1, U705.7 (-VOUT)
- new net ISO_EN: U704.3 (ON)
- new net PROT_EN: U702.3 (EN)
- new net VBUS: JP702.1 (A)
- no-connect marks 0 -> 1
Other:
- note added: "12V, 390mA"
- note added: "5V, 130mA"
- note added: "5V, 200mA"
- note added: "5V, 255mA"
- note added: "5V, 600mA"
- note added: "Expect up to 22mV drop, 5mW dissipation"
- note added: "Power Regulation"
- note removed: "3.3V, 0.15A"
- note removed: "5V, 0.5A"
- note removed: "Expect 0.25W dissipation"
- note removed: "Expect 0.65W dissipation"
- note removed: "Tantalum recommended"
- company: (none) -> LHR Solar
- title: (none) -> Sunscatter MPPT

Commit message: HW sch changes, further layout progression
Parts:
- removed C701: 100n, Resistor_SMD:R_0402_1005Metric, symbol Device:C_Small
- removed J702: PWR Header, footprints:molex_microfit_43650_0227, symbol molex_microfit_43650_0227:43650-0227
- removed JP703: Jumper_2_Bridged, Connector_PinHeader_2.54mm:PinHeader_1x02_P2.54mm_Vertical, symbol Jumper:Jumper_2_Bridged
- added C301: 100n, Resistor_SMD:R_0402_1005Metric, symbol Device:C_Small
- J301: renamed from J701; value PWR Header -> CAR PWR
- TP301: renamed from TP701; footprint TestPoint:TestPoint_Keystone_5000-5004_Miniature -> TestPoint:TestPoint_Pad_D1.5mm; Cost 0.31 -> (none); Distributor Mouser -> (none); Manufacturer Keystone Electronics -> (none); Notes Red (Logic Power) -> (none); P/N 5000 -> (none)
- TP302: renamed from TP705; footprint TestPoint:TestPoint_Keystone_5000-5004_Miniature -> TestPoint:TestPoint_Pad_D1.5mm; Cost 0.37 -> (none); Distributor Mouser -> (none); Manufacturer Keystone Electronics -> (none); Notes Black (Logic Ground) -> (none); P/N 5001 -> (none)
- TP303: renamed from TP702; footprint TestPoint:TestPoint_Keystone_5000-5004_Miniature -> TestPoint:TestPoint_Pad_D1.5mm; Cost 0.31 -> (none); Distributor Mouser -> (none); Manufacturer Keystone Electronics -> (none); Notes Red (Logic Power) -> (none); P/N 5000 -> (none)
- TP304: renamed from TP703; footprint TestPoint:TestPoint_Keystone_5000-5004_Miniature -> TestPoint:TestPoint_Pad_D1.5mm; Cost 0.31 -> (none); Distributor Mouser -> (none); Manufacturer Keystone Electronics -> (none); Notes Red (Logic Power) -> (none); P/N 5000 -> (none)
- TP305: renamed from TP704; footprint TestPoint:TestPoint_Keystone_5000-5004_Miniature -> TestPoint:TestPoint_Pad_D1.5mm; Cost 0.31 -> (none); Distributor Mouser -> (none); Manufacturer Keystone Electronics -> (none); Notes Red (Logic Power) -> (none); P/N 5000 -> (none)
- TP306: renamed from TP706; footprint TestPoint:TestPoint_Keystone_5000-5004_Miniature -> TestPoint:TestPoint_Pad_D1.5mm; Cost 0.31 -> (none); Distributor Mouser -> (none); Manufacturer Keystone Electronics -> (none); Notes Red (Logic Power) -> (none); P/N 5000 -> (none)
- TP307: renamed from TP707; footprint TestPoint:TestPoint_Keystone_5000-5004_Miniature -> TestPoint:TestPoint_Pad_D1.5mm; Cost 0.37 -> (none); Distributor Mouser -> (none); Manufacturer Keystone Electronics -> (none); Notes Brown (Power Path Ground) -> (none); P/N 5115 -> (none)
- renumbered C702 to C302, C703 to C303, C704 to C304, C705 to C305, C706 to C306, C707 to C307, C708 to C308, C709 to C309, C710 to C310, C711 to C311, C712 to C312, C713 to C313, C714 to C314, D701 to D301, D702 to D302, D703 to D303, D704 to D304, D705 to D305, JP701 to JP301, JP702 to JP302, L701 to L301, L702 to L302, Q701 to Q301, R701 to R301, R702 to R302, R703 to R303, R704 to R304, R705 to R305, U701 to U301, U702 to U302, U703 to U303, U704 to U304, U705 to U305, U706 to U306
Connections:
- net GND: now also C301.1
- net at C302.1, D301.2 (A2), J301.1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: now also C301.2
Other:
- moved on the sheet: C310, C312, C313, D304, D305, JP301, JP302, R304, R305, TP302, U306
